Commit message: first update attempt

File: urdf/pioneer-lx-devil.urdf (robot description, URDF)
Before this commit: robot pioneer-lx-devil, 39 links, 38 joints
Links:
- link base_link: geometry collision box size=0.697 0.5 0.35; visual mesh filename=package://amr-ros-config/meshes/pioneer-lx/pioneer-lx_visua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 scale=0.001 0.001 0.001
- link plinth: geometry collision mesh filename=package://amr-ros-config/meshes/pioneer-lx/pioneer-lx-plint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 scale=0.001 0.001 0.001; visual mesh filename=package://amr-ros-config/meshes/pioneer-lx/pioneer-lx-plint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 scale=0.001 0.001 0.001

File: urdf/pioneer-lx-devil.urdf.xacro (robot description, xacro)
@@ -24,5 +24,5 @@
     <visual name="base_link_visual">
       <geometry name="base_link_visual_geom">
-        <mesh filename="package://amr_robots_description/meshes/pioneer-lx/pioneer-lx_visual.stl" scale="0.001 0.001 0.001" />
+        <mesh filename="package://amr-ros-config/meshes/pioneer-lx/pioneer-lx_visual.stl" scale="0.001 0.001 0.001" />
         <!-- box size="0.697 0.5 0.333" / -->
       </geometry>
@@ -137,5 +137,5 @@
     <visual name="plinth_visual">
       <geometry name="plinth_visual_geom">
-        <mesh filename="package://amr_robots_description/meshes/pioneer-lx/pioneer-lx-plinth.stl" scale="0.001 0.001 0.001" />
+        <mesh filename="package://amr-ros-config/meshes/pioneer-lx/pioneer-lx-plinth.stl" scale="0.001 0.001 0.001" />
         <!-- box size="0.18 0.2476 0.99" / -->
       </geometry>
@@ -146,5 +146,5 @@
     <collision name="plinth_collision">
       <geometry name="plinth_collision_geom">
-        <mesh filename="package://amr_robots_description/meshes/pioneer-lx/pioneer-lx-plinth.stl" scale="0.001 0.001 0.001" />
+        <mesh filename="package://amr-ros-config/meshes/pioneer-lx/pioneer-lx-plinth.stl" scale="0.001 0.001 0.001" />
         <!-- box size="0.18 0.2476 0.99" / -->
         <origin xyz="-0.02 0 0.867" />

File: urdf/pioneer-lx.urdf (robot description, URDF)
Before this commit: robot pioneer-lx, 4 links, 3 joints
Links:
- link base_link: geometry collision box size=0.7 0.5 0.35; visual mesh filename=package://amr-ros-config/meshes/pioneer-lx/pioneer-lx_visua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 scale=0.001 0.001 0.001

File: urdf/pioneer-lx.urdf.xacro (robot description, xacro)
@@ -1,26 +1,21 @@
-<?xml version="1.0" ?>
-<!-- =================================================================================== -->
-<!-- |    This document was autogenerated by xacro from pioneer-lx.urdf.xacro          | -->
-<!-- |    EDITING THIS FILE BY HAND IS NOT RECOMMENDED                                 | -->
-<!-- =================================================================================== -->
+<?xml version="1.0"?>
 <robot name="pioneer-lx" xmlns:xacro="http://ros.org/wiki/xacro">
   <link name="base_link">
     <!-- base_link origin point is center of rotation, on the floor. -->
     <inertial>
-      <mass value="57.8"/>
-      <!-- 60 kg minus each wheel -->
-      <inertia ixx="1" ixy="0" ixz="0" iyy="1" iyz="0" izz="1"/>
+      <mass value="57.8" /> <!-- 60 kg minus each wheel -->
+      <inertia ixx="1" ixy="0" ixz="0" iyy="1" iyz="0" izz="1" />
     </inertial>
     <visual>
       <geometry name="base_link_visual_geom">
-        <mesh filename="package://amr_robots_description/meshes/pioneer-lx/pioneer-lx_visual.stl" scale="0.001 0.001 0.001"/>
+        <mesh filename="package://amr-ros-config/meshes/pioneer-lx/pioneer-lx_visual.stl" scale="0.001 0.001 0.001" />
       </geometry>
-      <origin rpy="0 0 1.570796" xyz="0 0 0.0"/>
+      <origin xyz="0 0 0.0" rpy="0 0 1.570796" />
     </visual>
     <collision name="base_link_collision">
       <geometry name="base_link_collision_geom">
-        <box size="0.7 0.5 0.35"/>
+        <box size="0.7 0.5 0.35" />
       </geometry>
-      <origin rpy="0 0 0" xyz="0 0 0.2"/>
+      <origin xyz="0 0 0.2" rpy="0 0 0" />
     </collision>
   </link>
@@ -28,9 +23,8 @@
   <link name="r_wheel">
     <inertial>
-      <mass value="1.1"/>
-      <!-- kg -->
-      <inertia ixx="0.02" ixy="0" ixz="0" iyy="0.02" iyz="0" izz="0.01"/>
+      <mass value="1.1" />   <!-- kg -->
+      <inertia ixx="0.02" ixy="0" ixz="0" iyy="0.02" iyz="0" izz="0.01" />
     </inertial>
-    <!--
+<!--
 TODO separate out pioner lx wheels in visual model
     <visual>
@@ -43,7 +37,7 @@
     <collision name="r_wheel_collision">
       <geometry name="r_wheel_collision_geom">
-        <cylinder length="0.05" radius="0.100"/>
+        <cylinder radius="0.100" length="0.05" />
       </geometry>
-      <origin rpy="1.570796 0 0"/>
+      <origin rpy="1.570796 0 0" />
     </collision>
   </link>
@@ -51,9 +45,8 @@
   <link name="l_wheel">
     <inertial>
-      <mass value="1.1"/>
-      <!-- kg -->
-      <inertia ixx="0.02" ixy="0" ixz="0" iyy="0.02" iyz="0" izz="0.01"/>
+      <mass value="1.1" />   <!-- kg -->
+      <inertia ixx="0.02" ixy="0" ixz="0" iyy="0.02" iyz="0" izz="0.01" />
     </inertial>
-    <!--
+<!--
     <visual>
       <geometry name="l_wheel_dumb_visual_geom">
@@ -65,19 +58,19 @@
     <collision name="l_wheel_collision">
       <geometry name="l_wheel_collision_geom">
-        <cylinder length="0.05" radius="0.100"/>
+        <cylinder radius="0.100" length="0.05" />
       </geometry>
-      <origin rpy="1.570796 0 0"/>
+      <origin rpy="1.570796 0 0" />
     </collision>
   </link>
   <!-- joints -->
   <joint name="r_wheel_joint" type="continuous">
-    <origin rpy="0 0 0" xyz="0 0.2 0.1"/>
-    <parent link="base_link"/>
-    <child link="r_wheel"/>
+    <origin xyz="0 0.2 0.1" rpy="0 0 0" />
+    <parent link="base_link" />
+    <child link="r_wheel" />
   </joint>
   <joint name="l_wheel_joint" type="continuous">
-    <origin rpy="0 0 0" xyz="0 -0.2 0.1"/>
-    <parent link="base_link"/>
-    <child link="l_wheel"/>
+    <origin xyz="0 -0.2 0.1" rpy="0 0 0" />
+    <parent link="base_link" />
+    <child link="l_wheel" />
   </joint>
   <!-- pioneer lx deck -->
@@ -85,23 +78,23 @@
     <visual>
       <geometry name="deck_visual_geom">
-        <box size="0.407 0.437 0.076"/>
+        <box size="0.407 0.437 0.076" />
       </geometry>
       <material name="lx_deck_mat">
-        <color rgba="0.1 0.1 0.1 1"/>
+        <color rgba="0.1 0.1 0.1 1" />
       </material>
     </visual>
     <collision name="deck_collision">
       <geometry name="deck_collision_geom">
-        <box size="0.407 0.437 0.076"/>
+        <box size="0.407 0.437 0.076" />
       </geometry>
     </collision>
   </link>
   <joint name="deck_joint" type="fixed">
-    <origin rpy="0 0 0" xyz="0.075 0 0.410"/>
-    <parent link="base_link"/>
-    <child link="deck"/>
+    <origin xyz="0.075 0 0.410" rpy="0 0 0" />
+    <parent link="base_link" />
+    <child link="deck" />
   </joint>
   <gazebo>
-    <plugin filename="libgazebo_ros_diff_drive.so" name="differential_drive_controller">
+    <plugin name="differential_drive_controller" filename="libgazebo_ros_diff_drive.so">
       <alwaysOn>true</alwaysOn>
       <updateRate>100</updateRate>
@@ -117,5 +110,5 @@
       <odometryFrame>odom</odometryFrame>
     </plugin>
-    <!-- TODO include P3D (ground truth) plugin -->
+  <!-- TODO include P3D (ground truth) plugin -->
   </gazebo>
 </robot>

File: urdf/pioneer3at.urdf (robot description, URDF)
Before this commit: robot pioneer3at, 16 links, 15 joints
Links:
- link back_sonar: geometry visual mesh filename=package://amr-ros-config/meshes/p3at_meshes/back_sonar.stl
- link base_link: geometry collision mesh filename=package://amr-ros-config/meshes/p3at_meshes/chassis.stl; visual mesh filename=package://amr-ros-config/meshes/p3at_meshes/chassis.stl
- link front_sonar: geometry visual mesh filename=package://amr-ros-config/meshes/p3at_meshes/front_sonar.stl
- link p3at_back_left_axle: geometry collision mesh filename=package://amr-ros-config/meshes/p3at_meshes/axle.stl; visual mesh filename=package://amr-ros-config/meshes/p3at_meshes/axle.stl
- link p3at_back_left_hub: geometry collision mesh filename=package://amr-ros-config/meshes/p3at_meshes/left_hubcap.stl; visual mesh filename=package://amr-ros-config/meshes/p3at_meshes/left_hubcap.stl
- link p3at_back_left_wheel: geometry collision cylinder length=0.075 radius=0.111; visual mesh filename=package://amr-ros-config/meshes/p3at_meshes/wheel.stl
- link p3at_back_right_axle: geometry collision mesh filename=package://amr-ros-config/meshes/p3at_meshes/axle.stl; visual mesh filename=package://amr-ros-config/meshes/p3at_meshes/axle.stl
- link p3at_back_right_hub: geometry collision mesh filename=package://amr-ros-config/meshes/p3at_meshes/right_hubcap.stl; visual mesh filename=package://amr-ros-config/meshes/p3at_meshes/right_hubcap.stl
- link p3at_back_right_wheel: geometry collision cylinder length=0.075 radius=0.111; visual mesh filename=package://amr-ros-config/meshes/p3at_meshes/wheel.stl
- link p3at_front_left_axle: geometry visual mesh filename=package://amr-ros-config/meshes/p3at_meshes/axle.stl
- link p3at_front_left_hub: geometry visual mesh filename=package://amr-ros-config/meshes/p3at_meshes/left_hubcap.stl
- link p3at_front_left_wheel: geometry collision cylinder length=0.075 radius=0.111; visual mesh filename=package://amr-ros-config/meshes/p3at_meshes/wheel.stl
- link p3at_front_right_axle: geometry visual mesh filename=package://amr-ros-config/meshes/p3at_meshes/axle.stl
- link p3at_front_right_hub: geometry visual mesh filename=package://amr-ros-config/meshes/p3at_meshes/right_hubcap.stl
- link p3at_front_right_wheel: geometry collision cylinder length=0.075 radius=0.111; visual mesh filename=package://amr-ros-config/meshes/p3at_meshes/wheel.stl
- link top_plate: geometry visual mesh filename=package://amr-ros-config/meshes/p3at_meshes/top.stl

File: urdf/pioneer3at.urdf.xacro (robot description, xacro)
@@ -24,5 +24,5 @@
 			<origin xyz="0 0 0.177" rpy="0 0 0"/>
 			<geometry name="pioneer_geom">
-				<mesh filename="package://amr_robots_description/meshes/p3at_meshes/chassis.stl"/>
+				<mesh filename="package://amr-ros-config/meshes/p3at_meshes/chassis.stl"/>
 			</geometry>
 			<material name="ChassisRed">
@@ -33,5 +33,5 @@
 			<origin xyz="0 0 0.177" rpy="0 0 0"/>
 				<geometry>
-					<mesh filename="package://amr_robots_description/meshes/p3at_meshes/chassis.stl"/>
+					<mesh filename="package://amr-ros-config/meshes/p3at_meshes/chassis.stl"/>
 				</geometry>
 		</collision>
@@ -52,5 +52,5 @@
 			<origin xyz="0 0 0" rpy="0 0 0"/>
 			<geometry name="pioneer_geom">
-				<mesh filename="package://amr_robots_description/meshes/p3at_meshes/top.stl"/>
+				<mesh filename="package://amr-ros-config/meshes/p3at_meshes/top.stl"/>
 			</geometry>
 			<material name="TopBlack">
@@ -78,5 +78,5 @@
 			<origin xyz="0 0 0" rpy="0 0 0"/>
 			<geometry name="pioneer_geom">
-				<mesh filename="package://amr_robots_description/meshes/p3at_meshes/front_sonar.stl"/>
+				<mesh filename="package://amr-ros-config/meshes/p3at_meshes/front_sonar.stl"/>
 			</geometry>
 			<material name="SonarYellow">
@@ -103,5 +103,5 @@
 			<origin xyz="0 0 0" rpy="0 0 0"/>
 			<geometry name="pioneer_geom">
-				<mesh filename="package://amr_robots_description/meshes/p3at_meshes/back_sonar.stl"/>
+				<mesh filename="package://amr-ros-config/meshes/p3at_meshes/back_sonar.stl"/>
 			</geometry>
 			<material name="SonarYellow">
@@ -130,5 +130,5 @@
 		<origin xyz="0 0 0" rpy="0 0 0"/>
 		<geometry name="pioneer_geom">
-			<mesh filename="package://amr_robots_description/meshes/p3at_meshes/axle.stl"/>
+			<mesh filename="package://amr-ros-config/meshes/p3at_meshes/axle.stl"/>
 		</geometry>
 		<material name="AxleGrey">
@@ -155,5 +155,5 @@
 		<origin xyz="0 0 0" rpy="0 0 0"/>
 		<geometry name="pioneer_geom">
-			<mesh filename="package://amr_robots_description/meshes/p3at_meshes/${side}_hubcap.stl"/>
+			<mesh filename="package://amr-ros-config/meshes/p3at_meshes/${side}_hubcap.stl"/>
 		</geometry>
 		<material name="HubcapYellow">
@@ -180,5 +180,5 @@
 		<origin xyz="0 0 0" rpy="0 0 0"/>
 		<geometry name="pioneer_geom">
-			<mesh filename="package://amr_robots_description/meshes/p3at_meshes/wheel.stl"/>
+			<mesh filename="package://amr-ros-config/meshes/p3at_meshes/wheel.stl"/>
 		</geometry>
 		<material name="WheelBlack">
@@ -189,5 +189,5 @@
 		<origin xyz="0 0 0" rpy="${-3.1415927/2} 0 0"/>
 		<geometry>
-	    <!--mesh filename="package://amr_robots_description/meshes/p3at_meshes/wheel.stl"/-->
+	    <!--mesh filename="package://amr-ros-config/meshes/p3at_meshes/wheel.stl"/-->
 	    <cylinder radius="0.111" length="0.075"/>
 		</geometry>
@@ -217,5 +217,5 @@
 		<origin xyz="0 0 0" rpy="0 0 0"/>
 		<geometry name="pioneer_geom">
-			<mesh filename="package://amr_robots_description/meshes/p3at_meshes/axle.stl"/>
+			<mesh filename="package://amr-ros-config/meshes/p3at_meshes/axle.stl"/>
 		</geometry>
 		<material name="AxleGrey">
@@ -226,5 +226,5 @@
 		<origin xyz="0 0 0" rpy="0 0 0"/>
 		<geometry>
-			<mesh filename="package://amr_robots_description/meshes/p3at_meshes/axle.stl"/>
+			<mesh filename="package://amr-ros-config/meshes/p3at_meshes/axle.stl"/>
 		</geometry>
 	</collision>
@@ -248,5 +248,5 @@
 		<origin xyz="0 0 0" rpy="0 0 0"/>
 		<geometry name="pioneer_geom">
-			<mesh filename="package://amr_robots_description/meshes/p3at_meshes/${side}_hubcap.stl"/>
+			<mesh filename="package://amr-ros-config/meshes/p3at_meshes/${side}_hubcap.stl"/>
 		</geometry>
 		<material name="HubcapYellow"/>
@@ -255,5 +255,5 @@
 		<origin xyz="0 0 0" rpy="0 0 0"/>
 		<geometry>
-			<mesh filename="package://amr_robots_description/meshes/p3at_meshes/${side}_hubcap.stl"/>
+			<mesh filename="package://amr-ros-config/meshes/p3at_meshes/${side}_hubcap.stl"/>
 		</geometry>
 	</collision>
@@ -278,5 +278,5 @@
 		<origin xyz="0 0 0" rpy="0 0 0"/>
 		<geometry name="pioneer_geom">
-			<mesh filename="package://amr_robots_description/meshes/p3at_meshes/wheel.stl"/>
+			<mesh filename="package://amr-ros-config/meshes/p3at_meshes/wheel.stl"/>
 		</geometry>
 		<material name="WheelBlack"/>
@@ -285,5 +285,5 @@
 		<origin xyz="0 0 0" rpy="${-3.1415927/2} 0 0"/>
 		<geometry>
-	    <!--mesh filename="package://amr_robots_description/meshes/p3at_meshes/wheel.stl"/-->
+	    <!--mesh filename="package://amr-ros-config/meshes/p3at_meshes/wheel.stl"/-->
 	    <cylinder radius="0.111" length="0.075"/>
 		</geometry>

File: urdf/pioneer3at_body.xacro (robot description, xacro)
@@ -17,5 +17,5 @@
 			<origin xyz="0 0 0.177" rpy="0 0 0"/>
 			<geometry name="pioneer_geom">
-				<mesh filename="package://amr_robots_description/meshes/p3at_meshes/chassis.stl"/>
+				<mesh filename="package://amr-ros-config/meshes/p3at_meshes/chassis.stl"/>
 			</geometry>
 			<material name="ChassisRed">
@@ -26,5 +26,5 @@
 			<origin xyz="0 0 0.177" rpy="0 0 0"/>
 				<geometry>
-					<mesh filename="package://amr_robots_description/meshes/p3at_meshes/chassis.stl"/>
+					<mesh filename="package://amr-ros-config/meshes/p3at_meshes/chassis.stl"/>
 				</geometry>
 		</collision>
@@ -45,5 +45,5 @@
 			<origin xyz="0 0 0" rpy="0 0 0"/>
 			<geometry name="pioneer_geom">
-				<mesh filename="package://amr_robots_description/meshes/p3at_meshes/top.stl"/>
+				<mesh filename="package://amr-ros-config/meshes/p3at_meshes/top.stl"/>
 			</geometry>
 			<material name="TopBlack">
@@ -71,5 +71,5 @@
 			<origin xyz="0 0 0" rpy="0 0 0"/>
 			<geometry name="pioneer_geom">
-				<mesh filename="package://amr_robots_description/meshes/p3at_meshes/front_sonar.stl"/>
+				<mesh filename="package://amr-ros-config/meshes/p3at_meshes/front_sonar.stl"/>
 			</geometry>
 			<material name="SonarYellow">
@@ -96,5 +96,5 @@
 			<origin xyz="0 0 0" rpy="0 0 0"/>
 			<geometry name="pioneer_geom">
-				<mesh filename="package://amr_robots_description/meshes/p3at_meshes/back_sonar.stl"/>
+				<mesh filename="package://amr-ros-config/meshes/p3at_meshes/back_sonar.stl"/>
 			</geometry>
 			<material name="SonarYellow">
@@ -123,5 +123,5 @@
 		<origin xyz="0 0 0" rpy="0 0 0"/>
 		<geometry name="pioneer_geom">
-			<mesh filename="package://amr_robots_description/meshes/p3at_meshes/axle.stl"/>
+			<mesh filename="package://amr-ros-config/meshes/p3at_meshes/axle.stl"/>
 		</geometry>
 		<material name="AxleGrey">
@@ -148,5 +148,5 @@
 		<origin xyz="0 0 0" rpy="0 0 0"/>
 		<geometry name="pioneer_geom">
-			<mesh filename="package://amr_robots_description/meshes/p3at_meshes/${suffix}_hubcap.stl"/>
+			<mesh filename="package://amr-ros-config/meshes/p3at_meshes/${suffix}_hubcap.stl"/>
 		</geometry>
 		<material name="HubcapYellow">
@@ -173,5 +173,5 @@
 		<origin xyz="0 0 0" rpy="0 0 0"/>
 		<geometry name="pioneer_geom">
-			<mesh filename="package://amr_robots_description/meshes/p3at_meshes/wheel.stl"/>
+			<mesh filename="package://amr-ros-config/meshes/p3at_meshes/wheel.stl"/>
 		</geometry>
 		<material name="WheelBlack">
@@ -182,5 +182,5 @@
 		<origin xyz="0 0 0" rpy="${-3.1415927/2} 0 0"/>
 		<geometry>
-	    <!--mesh filename="package://amr_robots_description/meshes/p3at_meshes/wheel.stl"/-->
+	    <!--mesh filename="package://amr-ros-config/meshes/p3at_meshes/wheel.stl"/-->
 	    <cylinder radius="0.111" length="0.075"/>
 		</geometry>
@@ -210,5 +210,5 @@
 		<origin xyz="0 0 0" rpy="0 0 0"/>
 		<geometry name="pioneer_geom">
-			<mesh filename="package://amr_robots_description/meshes/p3at_meshes/axle.stl"/>
+			<mesh filename="package://amr-ros-config/meshes/p3at_meshes/axle.stl"/>
 		</geometry>
 		<material name="AxleGrey">
@@ -219,5 +219,5 @@
 		<origin xyz="0 0 0" rpy="0 0 0"/>
 		<geometry>
-			<mesh filename="package://amr_robots_description/meshes/p3at_meshes/axle.stl"/>
+			<mesh filename="package://amr-ros-config/meshes/p3at_meshes/axle.stl"/>
 		</geometry>
 	</collision>
@@ -241,5 +241,5 @@
 		<origin xyz="0 0 0" rpy="0 0 0"/>
 		<geometry name="pioneer_geom">
-			<mesh filename="package://amr_robots_description/meshes/p3at_meshes/${suffix}_hubcap.stl"/>
+			<mesh filename="package://amr-ros-config/meshes/p3at_meshes/${suffix}_hubcap.stl"/>
 		</geometry>
 		<material name="HubcapYellow"/>
@@ -248,5 +248,5 @@
 		<origin xyz="0 0 0" rpy="0 0 0"/>
 		<geometry>
-			<mesh filename="package://amr_robots_description/meshes/p3at_meshes/${suffix}_hubcap.stl"/>
+			<mesh filename="package://amr-ros-config/meshes/p3at_meshes/${suffix}_hubcap.stl"/>
 		</geometry>
 	</collision>
@@ -270,5 +270,5 @@
 		<origin xyz="0 0 0" rpy="0 0 0"/>
 		<geometry name="pioneer_geom">
-			<mesh filename="package://amr_robots_description/meshes/p3at_meshes/wheel.stl"/>
+			<mesh filename="package://amr-ros-config/meshes/p3at_meshes/wheel.stl"/>
 		</geometry>
 		<material name="WheelBlack"/>
@@ -277,5 +277,5 @@
 		<origin xyz="0 0 0" rpy="${-3.1415927/2} 0 0"/>
 		<geometry>
-	    <!--mesh filename="package://amr_robots_description/meshes/p3at_meshes/wheel.stl"/-->
+	    <!--mesh filename="package://amr-ros-config/meshes/p3at_meshes/wheel.stl"/-->
 	    <cylinder radius="0.111" length="0.075"/>
 		</geometry>

File: urdf/pioneer3dx.urdf (robot description, URDF)
Before this commit: robot pioneer3dx, 11 links, 10 joints
Links:
- link back_sonar: geometry visual mesh filename=package://amr-ros-config/meshes/p3dx_meshes/back_sonar.stl
- link base_link: geometry collision box size=0.01 0.01 0.01; visual mesh filename=package://amr-ros-config/meshes/p3dx_meshes/chassis.stl
- link caster_hubcap: geometry collision box size=0.05 0.05 0.05; visual mesh filename=package://amr-ros-config/meshes/p3dx_meshes/caster_hubcap.s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
- link caster_swivel: geometry visual mesh filename=package://amr-ros-config/meshes/p3dx_meshes/caster_swivel.s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
- link caster_wheel: geometry collision cylinder length=0.01 radius=0.0375; visual mesh filename=package://amr-ros-config/meshes/p3dx_meshes/caster_wheel.stl
- link front_sonar: geometry visual mesh filename=package://amr-ros-config/meshes/p3dx_meshes/front_sonar.stl
- link left_hub: geometry collision cylinder length=0.01 radius=0.09; visual mesh filename=package://amr-ros-config/meshes/p3dx_meshes/left_hubcap.stl
- link left_wheel: geometry visual mesh filename=package://amr-ros-config/meshes/p3dx_meshes/left_wheel.stl
- link right_hub: geometry collision cylinder length=0.01 radius=0.09; visual mesh filename=package://amr-ros-config/meshes/p3dx_meshes/right_hubcap.stl
- link right_wheel: geometry visual mesh filename=package://amr-ros-config/meshes/p3dx_meshes/right_wheel.stl
- link top_plate: geometry visual mesh filename=package://amr-ros-config/meshes/p3dx_meshes/top.stl
