Commit message: first update attempt

File: urdf/pioneer3dx.urdf.xacro (robot description, xacro)
@@ -5,6 +5,6 @@
 	xmlns:interface="http://playerstage.sourceforge.net/gazebo/xmlschema/#interface"
 	xmlns:xacro="http://ros.org/wiki/xacro">
-  <!--<include filename="$(find amr_robots_description)/urdf/materials.xacro"/>-->
-  <xacro:include filename="$(find amr_robots_description)/urdf/pioneer3dx_wheel.xacro"/>
+  <!--<include filename="$(find amr-ros-config)/urdf/materials.xacro"/>-->
+  <xacro:include filename="$(find amr-ros-config)/urdf/pioneer3dx_wheel.xacro"/>
 <!-- Chassis -->
 	<link name="base_link">
@@ -20,5 +20,5 @@
 			<origin xyz="-0.045 0 0.148" rpy="0 0 0"/>
 			<geometry name="pioneer_geom">
-				<mesh filename="package://amr_robots_description/meshes/p3dx_meshes/chassis.stl"/>
+				<mesh filename="package://amr-ros-config/meshes/p3dx_meshes/chassis.stl"/>
 			</geometry>
 			<material name="ChassisRed">
@@ -44,5 +44,5 @@
 			<origin xyz="0 0 0" rpy="0 0 0"/>
 			<geometry name="pioneer_geom">
-				<mesh filename="package://amr_robots_description/meshes/p3dx_meshes/top.stl"/>
+				<mesh filename="package://amr-ros-config/meshes/p3dx_meshes/top.stl"/>
 			</geometry>
 			<material name="TopBlack">
@@ -71,5 +71,5 @@
 			<origin xyz="0 0 0" rpy="0 0 0"/>
 			<geometry name="pioneer_geom">
-				<mesh filename="package://amr_robots_description/meshes/p3dx_meshes/front_sonar.stl"/>
+				<mesh filename="package://amr-ros-config/meshes/p3dx_meshes/front_sonar.stl"/>
 			</geometry>
 			<material name="SonarYellow">
@@ -93,5 +93,5 @@
 	<link name="back_sonar">
 		<inertial>
-			<mass value="0"/>
+			<mass value="0.0001"/>
 			<origin xyz="0 0 0"/>
 			<inertia ixx="1" ixy="0" ixz="0"
@@ -101,5 +101,5 @@
 			<origin xyz="0 0 0" rpy="0 0 0"/>
 			<geometry name="pioneer_geom">
-				<mesh filename="package://amr_robots_description/meshes/p3dx_meshes/back_sonar.stl"/>
+				<mesh filename="package://amr-ros-config/meshes/p3dx_meshes/back_sonar.stl"/>
 			</geometry>
 			<material name="SonarYellow">
@@ -127,5 +127,5 @@
 		<origin xyz="0 0 0" rpy="0 0 0"/>
 		<geometry name="pioneer_geom">
-			<mesh filename="package://amr_robots_description/meshes/p3dx_meshes/caster_swivel.stl"/>
+			<mesh filename="package://amr-ros-config/meshes/p3dx_meshes/caster_swivel.stl"/>
 		</geometry>
 		<material name="caster_swivel">
@@ -148,5 +148,5 @@
 		<origin xyz="0 0 0" rpy="0 0 0"/>
 		<geometry name="pioneer_geom">
-			<mesh filename="package://amr_robots_description/meshes/p3dx_meshes/caster_hubcap.stl"/>
+			<mesh filename="package://amr-ros-config/meshes/p3dx_meshes/caster_hubcap.stl"/>
 		</geometry>
 		<material name="caster_swivel">
@@ -183,5 +183,5 @@
 		<origin xyz="0 0 0" rpy="0 0 0"/>
 		<geometry name="pioneer_geom">
-			<mesh filename="package://amr_robots_description/meshes/p3dx_meshes/caster_wheel.stl"/>
+			<mesh filename="package://amr-ros-config/meshes/p3dx_meshes/caster_wheel.stl"/>
 		</geometry>
 		<material name="WheelBlack">
@@ -192,5 +192,5 @@
 		<origin xyz="0 0 0" rpy="${-3.1415927/2.0} 0 0"/>
 		<geometry>
-			<!--<mesh filename="package://amr_robots_description/meshes/p3dx_meshes/caster_wheel.stl"/>-->
+			<!--<mesh filename="package://amr-ros-config/meshes/p3dx_meshes/caster_wheel.stl"/>-->
 			<cylinder radius="0.0375" length="0.01"/>
 		</geometry>
@@ -209,5 +209,5 @@
 			<origin xyz="0 0 0" rpy="0 0 0"/>
 			<geometry>
-				<mesh filename="package://amr_robots_description/meshes/p3dx_meshes/left_hubcap.stl"/>
+				<mesh filename="package://amr-ros-config/meshes/p3dx_meshes/left_hubcap.stl"/>
 			</geometry>
 			<material name="HubcapYellow">
@@ -218,5 +218,5 @@
 			<origin xyz="0 0 0" rpy="${-3.1415927/2.0} 0 0"/>
 			<geometry>
-				<!--<mesh filename="package://amr_robots_description/meshes/p3dx_meshes/caster_wheel.stl"/>-->
+				<!--<mesh filename="package://amr-ros-config/meshes/p3dx_meshes/caster_wheel.stl"/>-->
 				<cylinder radius="0.09" length="0.01"/>
 			</geometry>
@@ -233,5 +233,5 @@
 			<origin xyz="0 0 0" rpy="0 0 0"/>
 			<geometry>
-				<mesh filename="package://amr_robots_description/meshes/p3dx_meshes/left_wheel.stl"/>
+				<mesh filename="package://amr-ros-config/meshes/p3dx_meshes/left_wheel.stl"/>
 			</geometry>
 			<material name="WheelBlack">
@@ -252,5 +252,5 @@
 			<origin xyz="0 0 0" rpy="0 0 0"/>
 			<geometry>
-				<mesh filename="package://amr_robots_description/meshes/p3dx_meshes/right_hubcap.stl"/>
+				<mesh filename="package://amr-ros-config/meshes/p3dx_meshes/right_hubcap.stl"/>
 			</geometry>
 			<material name="HubcapYellow">
@@ -261,5 +261,5 @@
 		<origin xyz="0 0 0" rpy="${-3.1415927/2.0} 0 0"/>
 		<geometry>
-			<!--<mesh filename="package://amr_robots_description/meshes/p3dx_meshes/caster_wheel.stl"/>-->
+			<!--<mesh filename="package://amr-ros-config/meshes/p3dx_meshes/caster_wheel.stl"/>-->
 			<cylinder radius="0.09" length="0.01"/>
 		</geometry>
@@ -279,5 +279,5 @@
 			<origin xyz="0 0 0" rpy="0 0 0"/>
 			<geometry>
-				<mesh filename="package://amr_robots_description/meshes/p3dx_meshes/right_wheel.stl"/>
+				<mesh filename="package://amr-ros-config/meshes/p3dx_meshes/right_wheel.stl"/>
 			</geometry>
 			<material name="WheelBlack">

File: urdf/pioneer3dx_body.xacro (robot description, xacro)
@@ -6,5 +6,5 @@
 	   xmlns:xacro="http://ros.org/wiki/xacro"
 	   >
-	<xacro:include filename="$(find amr_robots_description)/urdf/pioneer3dx_wheel.xacro"/>
+	<xacro:include filename="$(find amr-ros-config)/urdf/pioneer3dx_wheel.xacro"/>
 	<!-- Chassis description -->
 	<link name="base_link">
@@ -21,5 +21,5 @@
 			<origin xyz="-0.045 0 0.148" rpy="0 0 0"/>
 			<geometry name="pioneer_geom">
-				<mesh filename="package://amr_robots_description/meshes/p3dx_meshes/chassis.stl"/>
+				<mesh filename="package://amr-ros-config/meshes/p3dx_meshes/chassis.stl"/>
 			</geometry>
 			<material name="ChassisRed">
@@ -30,5 +30,5 @@
 			<origin xyz="-0.045 0 0.148" rpy="0 0 0"/>
 				<geometry>
-					<mesh filename="package://amr_robots_description/meshes/p3at_meshes/chassis.stl"/>
+					<mesh filename="package://amr-ros-config/meshes/p3at_meshes/chassis.stl"/>
 				</geometry>
 		</collision>
@@ -48,5 +48,5 @@
 			<origin xyz="0 0 0" rpy="0 0 0"/>
 			<geometry name="pioneer_geom">
-				<mesh filename="package://amr_robots_description/meshes/p3dx_meshes/top.stl"/>
+				<mesh filename="package://amr-ros-config/meshes/p3dx_meshes/top.stl"/>
 			</geometry>
 			<material name="TopBlack">
@@ -82,5 +82,5 @@
 		<origin xyz="0 0 0" rpy="0 0 0"/>
 		<geometry name="pioneer_geom">
-			<mesh filename="package://amr_robots_description/meshes/p3dx_meshes/swivel.stl"/>
+			<mesh filename="package://amr-ros-config/meshes/p3dx_meshes/swivel.stl"/>
 		</geometry>
 		<material name="swivel">
@@ -103,5 +103,5 @@
 		<origin xyz="0 0 0" rpy="0 0 0"/>
 		<geometry name="pioneer_geom">
-			<mesh filename="package://amr_robots_description/meshes/p3dx_meshes/center_hubcap.stl"/>
+			<mesh filename="package://amr-ros-config/meshes/p3dx_meshes/center_hubcap.stl"/>
 		</geometry>
 		<material name="swivel">
@@ -138,5 +138,5 @@
 		<origin xyz="0 0 0" rpy="0 0 0"/>
 		<geometry name="pioneer_geom">
-			<mesh filename="package://amr_robots_description/meshes/p3dx_meshes/center_wheel.stl"/>
+			<mesh filename="package://amr-ros-config/meshes/p3dx_meshes/center_wheel.stl"/>
 		</geometry>
 		<material name="WheelBlack">
@@ -147,5 +147,5 @@
 		<origin xyz="0 0 0" rpy="${-3.1415927/2.0} 0 0"/>
 		<geometry>
-			<!--<mesh filename="package://amr_robots_description/meshes/p3dx_meshes/center_wheel.stl"/>-->
+			<!--<mesh filename="package://amr-ros-config/meshes/p3dx_meshes/center_wheel.stl"/>-->
 			<cylinder radius="0.0375" length="0.01"/>
 		</geometry>
@@ -164,5 +164,5 @@
 			<origin xyz="0 0 0" rpy="0 0 0"/>
 			<geometry>
-				<mesh filename="package://amr_robots_description/meshes/p3dx_meshes/left_hubcap.stl"/>
+				<mesh filename="package://amr-ros-config/meshes/p3dx_meshes/left_hubcap.stl"/>
 			</geometry>
 			<material name="HubcapYellow">
@@ -173,5 +173,5 @@
 			<origin xyz="0 0 0" rpy="${-3.1415927/2.0} 0 0"/>
 			<geometry>
-				<!--<mesh filename="package://amr_robots_description/meshes/p3dx_meshes/center_wheel.stl"/>-->
+				<!--<mesh filename="package://amr-ros-config/meshes/p3dx_meshes/center_wheel.stl"/>-->
 				<cylinder radius="0.09" length="0.01"/>
 			</geometry>
@@ -188,5 +188,5 @@
 			<origin xyz="0 0 0" rpy="0 0 0"/>
 			<geometry>
-				<mesh filename="package://amr_robots_description/meshes/p3dx_meshes/left_wheel.stl"/>
+				<mesh filename="package://amr-ros-config/meshes/p3dx_meshes/left_wheel.stl"/>
 			</geometry>
 			<material name="WheelBlack">
@@ -207,5 +207,5 @@
 			<origin xyz="0 0 0" rpy="0 0 0"/>
 			<geometry>
-				<mesh filename="package://amr_robots_description/meshes/p3dx_meshes/right_hubcap.stl"/>
+				<mesh filename="package://amr-ros-config/meshes/p3dx_meshes/right_hubcap.stl"/>
 			</geometry>
 			<material name="HubcapYellow">
@@ -216,5 +216,5 @@
 		<origin xyz="0 0 0" rpy="${-3.1415927/2.0} 0 0"/>
 		<geometry>
-			<!--<mesh filename="package://amr_robots_description/meshes/p3dx_meshes/center_wheel.stl"/>-->
+			<!--<mesh filename="package://amr-ros-config/meshes/p3dx_meshes/center_wheel.stl"/>-->
 			<cylinder radius="0.09" length="0.01"/>
 		</geometry>
@@ -234,5 +234,5 @@
 			<origin xyz="0 0 0" rpy="0 0 0"/>
 			<geometry>
-				<mesh filename="package://amr_robots_description/meshes/p3dx_meshes/right_wheel.stl"/>
+				<mesh filename="package://amr-ros-config/meshes/p3dx_meshes/right_wheel.stl"/>
 			</geometry>
 			<material name="WheelBlack">
@@ -260,5 +260,5 @@
 			<origin xyz="0 0 0" rpy="0 0 0"/>
 			<geometry name="pioneer_geom">
-				<mesh filename="package://amr_robots_description/meshes/p3dx_meshes/front_sonar.stl"/>
+				<mesh filename="package://amr-ros-config/meshes/p3dx_meshes/front_sonar.stl"/>
 			</geometry>
 			<material name="SonarYellow">
@@ -285,5 +285,5 @@
 			<origin xyz="0 0 0" rpy="0 0 0"/>
 			<geometry name="pioneer_geom">
-				<mesh filename="package://amr_robots_description/meshes/p3dx_meshes/back_sonar.stl"/>
+				<mesh filename="package://amr-ros-config/meshes/p3dx_meshes/back_sonar.stl"/>
 			</geometry>
 			<material name="SonarYellow">

File: urdf/pioneer3dx_wheel.xacro (robot description, xacro)
@@ -6,5 +6,5 @@
   xmlns:xacro="http://ros.org/wiki/xacro"
   >
-  <!--<include filename="$(find amr_robots_description)/urdf/materials.xacro"/>-->
+  <!--<include filename="$(find amr-ros-config)/urdf/materials.xacro"/>-->
   <!-- Properties (Constants) -->
   <property name="M_PI" value="3.14159"/>
@@ -21,5 +21,5 @@
       <origin xyz="0 0 0" rpy="0 0 0"/>
       <geometry name="pioneer_geom">
-        <mesh filename="package://amr_robots_description/meshes/p3dx_meshes/${suffix}_wheel.stl"/>
+        <mesh filename="package://amr-ros-config/meshes/p3dx_meshes/${suffix}_wheel.stl"/>
       </geometry>
       <material name="WheelBlack">
@@ -30,5 +30,5 @@
       <origin xyz="0 0 0" rpy="${-3.1415927/2} 0 0"/>
       <geometry>
-        <!--<mesh filename="package://amr_robots_description/meshes/p3dx_meshes/${suffix}_wheel.stl"/>-->
+        <!--<mesh filename="package://amr-ros-config/meshes/p3dx_meshes/${suffix}_wheel.stl"/>-->
         <cylinder radius="0.09" length="0.01"/>
       </geometry>
@@ -51,5 +51,5 @@
     <origin xyz="0 0 0" rpy="0 0 0"/>
     <geometry name="pioneer_geom">
-      <mesh filename="package://amr_robots_description/meshes/p3dx_meshes/${suffix}_hubcap.stl"/>
+      <mesh filename="package://amr-ros-config/meshes/p3dx_meshes/${suffix}_hubcap.stl"/>
     </geometry>
     <material name="HubcapYellow">

File: urdf/seekurjr.urdf.xacro (robot description, xacro)
@@ -17,5 +17,5 @@
 			<origin xyz="0 0 0.177" rpy="0 0 0"/>
 			<geometry name="skj_geom">
-				<!-- mesh filename="package://amr_robots_description/meshes/seekurjr_meshes/body.stl"/ -->
+				<!-- mesh filename="package://amr-ros-config/meshes/seekurjr_meshes/body.stl"/ -->
         <box size="0.440 1.050 0.500" />
 			</geometry>
@@ -27,5 +27,5 @@
 			<origin xyz="0 0 0.177" rpy="0 0 0"/>
 				<geometry>
-					<!-- mesh filename="package://amr_robots_description/meshes/seekurjr_meshes/body_collision.stl"/ -->
+					<!-- mesh filename="package://amr-ros-config/meshes/seekurjr_meshes/body_collision.stl"/ -->
           <box size="0.440 1.050 0.500" />
 				</geometry>
@@ -46,5 +46,5 @@
         <origin xyz="0 0 0" rpy="-1.570795 0 0"/>
         <geometry name="skj_wheel_geom">
-          <!-- mesh filename="package://amr_robots_description/meshes/skj_meshes/wheel.stl"/ -->
+          <!-- mesh filename="package://amr-ros-config/meshes/skj_meshes/wheel.stl"/ -->
           <cylinder radius="0.2" length="0.2"/>
         </geometry>
