Commit message: ros2 fix

File: urdf/pioneer3dx.urdf.xacro (robot description, xacro)
@@ -1,318 +1,11 @@
 <?xml version="1.0"?>
-<robot name="pioneer3dx"
-	xmlns:sensor="http://playerstage.sourceforge.net/gazebo/xmlschema/#sensor"
-	xmlns:controller="http://playerstage.sourceforge.net/gazebo/xmlschema/#controller"
-	xmlns:interface="http://playerstage.sourceforge.net/gazebo/xmlschema/#interface"
-	xmlns:xacro="http://ros.org/wiki/xacro">
-  <!--<include filename="$(find amr-ros-config)/urdf/materials.xacro"/>-->
-  <xacro:include filename="$(find amr-ros-config)/urdf/pioneer3dx_wheel.xacro"/>
-<!-- Chassis -->
-	<link name="base_link">
-		<inertial>
-			<mass value="3.5"/>
-			<!--<origin xyz="-0.025 0 -0.223"/>-->
-			<origin xyz="0 0 0"/>
-			<inertia ixx="1" ixy="0" ixz="0"
-				 iyy="1" iyz="0"
-				 izz="1"/>
-		</inertial>
-		<visual>
-			<origin xyz="-0.045 0 0.148" rpy="0 0 0"/>
-			<geometry name="pioneer_geom">
-				<mesh filename="package://amr-ros-config/meshes/p3dx_meshes/chassis.stl"/>
-			</geometry>
-			<material name="ChassisRed">
-				<color rgba="0.851 0.0 0.0 1.0"/>
-			</material>
-		</visual>
-		<collision>
-			<origin xyz="0 0 0" rpy="0 0 0"/>
-				<geometry>
-					<box size="0.01 0.01 0.01"/>
-				</geometry>
-		</collision>
-	</link>
-	<link name="top_plate">
-		<inertial>
-			<mass value="0.01"/>
-			<origin xyz="0 0 0"/>
-			<inertia ixx="1" ixy="0" ixz="0"
-				 iyy="1" iyz="0"
- 				izz="1"/>
-		</inertial>
-		<visual>
-			<origin xyz="0 0 0" rpy="0 0 0"/>
-			<geometry name="pioneer_geom">
-				<mesh filename="package://amr-ros-config/meshes/p3dx_meshes/top.stl"/>
-			</geometry>
-			<material name="TopBlack">
-					<color rgba="0.038 0.038 0.038 1.0"/>
-			</material>
-		</visual>
-	</link>
-	<gazebo reference="top_plate">
-		<!-- material value="Gazebo/Black"/ -->
-		<material>Gazebo/Black</material>
-	</gazebo>
-    <joint name="base_top_joint" type="fixed">
-		<origin xyz="-0.045 0 0.234" rpy="0 0 0"/>
-		<axis xzy="0 0 1"/>
-		<parent link="base_link"/>
-		<child link="top_plate"/>
-	</joint>
-	<link name="front_sonar">
-		<inertial>
-			<mass value="0.0001"/>
-			<origin xyz="0 0 0"/>
-			<inertia ixx="1" ixy="0" ixz="0"
-				 iyy="1" iyz="0" izz="1"/>
-		</inertial>
-		<visual>
-			<origin xyz="0 0 0" rpy="0 0 0"/>
-			<geometry name="pioneer_geom">
-				<mesh filename="package://amr-ros-config/meshes/p3dx_meshes/front_sonar.stl"/>
-			</geometry>
-			<material name="SonarYellow">
-				<color rgba="0.715 0.583 0.210 1.0"/>
-			</material>
-		</visual>
-	</link>
-	<gazebo reference="front_sonar">
-		<material value="Gazebo/Yellow"/>
-	</gazebo>
-	<joint name="base_front_joint" type="fixed">
-		<origin xyz="-0.198 0 0.208" rpy="0 0 0"/>
-		<parent link="base_link"/>
-		<child link="front_sonar"/>
-	</joint>
-	<joint name="base_back_joint" type="fixed">
-		<origin xyz="0.109 0 0.209" rpy="0 0 0"/>
-		<parent link="base_link"/>
-		<child link="back_sonar"/>
-	</joint>
-	<link name="back_sonar">
-		<inertial>
-			<mass value="0.0001"/>
-			<origin xyz="0 0 0"/>
-			<inertia ixx="1" ixy="0" ixz="0"
-				 iyy="1" iyz="0" izz="1"/>
-		</inertial>
-		<visual>
-			<origin xyz="0 0 0" rpy="0 0 0"/>
-			<geometry name="pioneer_geom">
-				<mesh filename="package://amr-ros-config/meshes/p3dx_meshes/back_sonar.stl"/>
-			</geometry>
-			<material name="SonarYellow">
-				<color rgba="0.715 0.583 0.210 1.0"/>
-			</material>
-		</visual>
-	</link>
-	<!-- Caster -->
-	<joint name="base_caster_swivel_joint" type="continuous">
-		<origin xyz="-0.185 0 0.055" rpy="0 0 0"/>
-		<anchor xyz="0 0 0"/>
-    	<limit effort="100" velocity="100" k_velocity="0" />
-    	<joint_properties damping="0.0" friction="0.0" />
-		<parent link="base_link"/>
-		<child link="caster_swivel"/>
-	</joint>
-	<link name="caster_swivel">
-		<inertial>
-			<mass value="0.1"/>
-			<origin xyz="0 0 0"/>
-			<inertia ixx="0.01" ixy="0" ixz="0"
-				 iyy="0.01" iyz="0" izz="0.01"/>
-  	 	</inertial>
-	<visual>
-		<origin xyz="0 0 0" rpy="0 0 0"/>
-		<geometry name="pioneer_geom">
-			<mesh filename="package://amr-ros-config/meshes/p3dx_meshes/caster_swivel.stl"/>
-		</geometry>
-		<material name="caster_swivel">
-			<color rgba="0.5 0.5 0.5 1"/>
-		</material>
-	</visual>
-	</link>
-	<gazebo reference="caster_swivel">
-		<material value="Gazebo/Grey"/>
-	</gazebo>
-<!-- Center Wheel + Hubcap -->
-	<link name="caster_hubcap">
-		<inertial>
-			<mass value="0.01"/>
-			<origin xyz="0 0 0"/>
-			<inertia ixx="0.012411765597" ixy="-0.000711733678" ixz="0.00050272983"
-				 iyy="0.015218160428" iyz="-0.000004273467" izz="0.011763977943"/>
-  	 	</inertial>
-	<visual>
-		<origin xyz="0 0 0" rpy="0 0 0"/>
-		<geometry name="pioneer_geom">
-			<mesh filename="package://amr-ros-config/meshes/p3dx_meshes/caster_hubcap.stl"/>
-		</geometry>
-		<material name="caster_swivel">
-			<color rgba="0.5 0.5 0.5 1"/>
-		</material>
-	</visual>
-	<collision>
-		<origin xyz="0 0 0" rpy="0 0 0"/>
-		<geometry>
-			<box size="0.05 0.05 0.05"/>
-		</geometry>
-	</collision>
-	</link>
-	<gazebo reference="caster_hubcap">
-		<material value="Gazebo/Grey"/>
-	</gazebo>
-	<joint name="caster_swivel_hubcap_joint" type="continuous">
-		<origin xyz="-0.026 0 -0.016" rpy="0 0 0"/>
-		<axis xyz="0 1 0"/>
-		<anchor xyz="0 0 0"/>
-    <limit effort="100" velocity="100" k_velocity="0" />
-    <joint_properties damping="0.0" friction="0.0" />
-	  <parent link="caster_swivel"/>
-		<child link="caster_wheel"/>
-	</joint>
-	<link name="caster_wheel">
-		<inertial>
-			<mass value="0.1"/>
-			<origin xyz="0 0 0"/>
-			<inertia ixx="0.012411765597" ixy="-0.000711733678" ixz="0.00050272983"
-				 iyy="0.015218160428" iyz="-0.000004273467" izz="0.011763977943"/>
-  	 	</inertial>
-	<visual>
-		<origin xyz="0 0 0" rpy="0 0 0"/>
-		<geometry name="pioneer_geom">
-			<mesh filename="package://amr-ros-config/meshes/p3dx_meshes/caster_wheel.stl"/>
-		</geometry>
-		<material name="WheelBlack">
-			<color rgba="0.117 0.117 0.117 1"/>
-		</material>
-	</visual>
-	<collision>
-		<origin xyz="0 0 0" rpy="${-3.1415927/2.0} 0 0"/>
-		<geometry>
-			<!--<mesh filename="package://amr-ros-config/meshes/p3dx_meshes/caster_wheel.stl"/>-->
-			<cylinder radius="0.0375" length="0.01"/>
-		</geometry>
-	</collision>
-	</link>
-	<gazebo reference="left_hub">
-		<material value="Gazebo/Yellow"/>
-	</gazebo>
-	<joint name="caster_wheel_joint" type="fixed">
-		<origin xyz="-0.0035 0 -0.001" rpy="0 0 0"/>
-		<parent link="caster_wheel"/>
-		<child link="caster_hubcap"/>
-	</joint>
-	<link name="left_hub">
-		<visual>
-			<origin xyz="0 0 0" rpy="0 0 0"/>
-			<geometry>
-				<mesh filename="package://amr-ros-config/meshes/p3dx_meshes/left_hubcap.stl"/>
-			</geometry>
-			<material name="HubcapYellow">
-				<color rgba="1.0 0.811 0.151 1.0"/>
-			</material>
-		</visual>
-		<collision>
-			<origin xyz="0 0 0" rpy="${-3.1415927/2.0} 0 0"/>
-			<geometry>
-				<!--<mesh filename="package://amr-ros-config/meshes/p3dx_meshes/caster_wheel.stl"/>-->
-				<cylinder radius="0.09" length="0.01"/>
-			</geometry>
-		</collision>
-	</link>
-	<joint name="left_hub_joint" type="fixed">
-		<origin xyz="0 0.15 0.08" rpy="0 0 0"/>
-		<parent link="base_link"/>
-		<child link="left_hub"/>
-		<axis xyz="0 1 0"/>
-	</joint>
-	<link name="left_wheel">
-		<visual>
-			<origin xyz="0 0 0" rpy="0 0 0"/>
-			<geometry>
-				<mesh filename="package://amr-ros-config/meshes/p3dx_meshes/left_wheel.stl"/>
-			</geometry>
-			<material name="WheelBlack">
-				<color rgba="0.117 0.117 0.117 1"/>
-			</material>
-		</visual>
-	</link>
-	<joint name="left_wheel_joint" type="fixed"> <!-- type="continuous" -->
-		<origin xyz="0 0 0" rpy="0 0 0"/>
-		<parent link="left_hub"/>
-		<child link="left_wheel"/>
-	</joint>
-	<gazebo reference="left_wheel_joint">
-		<material value="Gazebo/Black"/>
-	</gazebo>
-	<link name="right_hub">
-		<visual>
-			<origin xyz="0 0 0" rpy="0 0 0"/>
-			<geometry>
-				<mesh filename="package://amr-ros-config/meshes/p3dx_meshes/right_hubcap.stl"/>
-			</geometry>
-			<material name="HubcapYellow">
-				<color rgba="1.0 0.811 0.151 1.0"/>
-			</material>
-		</visual>
-		<collision>
-		<origin xyz="0 0 0" rpy="${-3.1415927/2.0} 0 0"/>
-		<geometry>
-			<!--<mesh filename="package://amr-ros-config/meshes/p3dx_meshes/caster_wheel.stl"/>-->
-			<cylinder radius="0.09" length="0.01"/>
-		</geometry>
-	</collision>
-	</link>
-	<gazebo reference="right_hub">
-		<material value="Gazebo/Yellow"/>
-	</gazebo>
-	<joint name="right_hub_joint" type="fixed">
-		<origin xyz="0 -0.15 0.08" rpy="0 0 0"/>
-		<parent link="base_link"/>
-		<child link="right_hub"/>
-		<axis xyz="0 1 0"/>
-	</joint>
-	<link name="right_wheel">
-		<visual>
-			<origin xyz="0 0 0" rpy="0 0 0"/>
-			<geometry>
-				<mesh filename="package://amr-ros-config/meshes/p3dx_meshes/right_wheel.stl"/>
-			</geometry>
-			<material name="WheelBlack">
-				<color rgba="0.117 0.117 0.117 1"/>
-			</material>
-		</visual>
-	</link>
-	<joint name="right_wheel_joint" type="fixed"> <!-- type="continuous" -->
-		<origin xyz="0 0 0" rpy="0 0 0"/>
-		<parent link="right_hub"/>
-		<child link="right_wheel"/>
-	</joint>
-	<gazebo reference="right_wheel_joint">
-		<material value="Gazebo/Black"/>
-	</gazebo>
-	<create>
-	<back_sonar parent="base_link"/>
-  	<top_plate  parent="base_link"/>
-  	</create>
-<gazebo>
-	<plugin name="differential_drive_controller" filename="libgazebo_ros_diff_drive.so">
-    <alwaysOn>true</alwaysOn>
-		<updateRate>100</updateRate>
-		<leftJoint>left_wheel_joint</leftJoint>
-		<rightJoint>right_wheel_joint</rightJoint>
-		<wheelSeparation>0.158</wheelSeparation>
-		<wheelDiameter>0.12</wheelDiameter>
-		<torque>5</torque>
-		<!-- interface:position name="position_iface_0"/ -->
-    <commandTopic>cmd_vel</commandTopic>
-    <robotBaseFrame>base_link</robotBaseFrame>
-    <odometryTopic>odom</odometryTopic>
-    <odometryFrame>odom</odometryFrame>
-	</plugin>
-  <!-- TODO include P3D (ground truth) plugin -->
-  <!-- XXX old urdf included a gazebo_ros_controller_manager plugin with a 1 second update rate -->
-</gazebo>
+<robot name="my_robot" xmlns:xacro="http://ros.org/wiki/xacro">
+  <!-- Include the Pioneer3DX macro -->
+  <xacro:include filename="$(find amr-ros-config)/urdf/pioneer3dx/pioneer3dx.urdf.xacro"/>
+  <!-- Create world link -->
+  <link name="world"/>
+  <!-- Instantiate the Pioneer3DX -->
+  <xacro:pioneer3dx prefix="pioneer3dx_robot" parent="world">
+    <origin xyz="0 0 0" rpy="0 0 0"/>
+  </xacro:pioneer3dx>
 </robot>

File: urdf/pioneer3dx/pioneer3dx_body.xacro (robot description, xacro)
@@ -6,5 +6,5 @@
 	   xmlns:xacro="http://ros.org/wiki/xacro"
 	   >
-	<xacro:include filename="$(find amr-ros-config)/urdf/pioneer3dx_wheel.xacro"/>
+	<xacro:include filename="$(find amr-ros-config)/urdf/pioneer3dx/pioneer3dx_wheel.xacro"/>
 	<!-- Chassis description -->
 	<link name="base_link">

Commit message: eliminated world frame dependency

File: urdf/pioneer3dx.urdf.xacro (robot description, xacro)
@@ -3,8 +3,6 @@
   <!-- Include the Pioneer3DX macro -->
   <xacro:include filename="$(find amr-ros-config)/urdf/pioneer3dx/pioneer3dx.urdf.xacro"/>
-  <!-- Create world link -->
-  <link name="world"/>
   <!-- Instantiate the Pioneer3DX -->
-  <xacro:pioneer3dx prefix="pioneer3dx_robot" parent="world">
+  <xacro:pioneer3dx prefix="pioneer3dx_robot">
     <origin xyz="0 0 0" rpy="0 0 0"/>
   </xacro:pioneer3dx>

File: urdf/pioneer3dx/pioneer3dx.urdf.xacro (robot description, xacro)
@@ -2,5 +2,5 @@
 <robot xmlns:xacro="http://ros.org/wiki/xacro">
 	<include filename="$(find amr-ros-config)/urdf/materials.xacro"/>
-	<xacro:macro name="pioneer3dx" params="prefix parent *origin">
+	<xacro:macro name="pioneer3dx" params="prefix *origin">
 		<xacro:include filename="$(find amr-ros-config)/urdf/pioneer3dx/pioneer3dx_wheel.xacro"/>
 		<!-- Base Link -->
@@ -27,10 +27,4 @@
 			</collision>
 		</link>
-		<!-- Connect to parent -->
-		<joint name="${prefix}base_joint" type="fixed">
-			<xacro:insert_block name="origin"/>
-			<parent link="${parent}"/>
-			<child link="${prefix}base_link"/>
-		</joint>
 		<!-- Top Plate -->
 		<link name="${prefix}top_plate">

Commit message: odom restored

File: urdf/pioneer3dx.urdf.xacro (robot description, xacro)
@@ -1,4 +1,4 @@
 <?xml version="1.0"?>
-<robot name="my_robot" xmlns:xacro="http://ros.org/wiki/xacro">
+<robot name="galax_robot" xmlns:xacro="http://ros.org/wiki/xacro">
   <!-- Include the Pioneer3DX macro -->
   <xacro:include filename="$(find amr-ros-config)/urdf/pioneer3dx/pioneer3dx.urdf.xacro"/>

File: urdf/pioneer3dx/pioneer3dx_sim.urdf.xacro (robot description, xacro)
@@ -15,7 +15,7 @@
 		<xacro:property name="top_plate_width" value="0.272"/>
 		<xacro:property name="top_plate_height" value="0.0052"/>
-		<xacro:property name="top_plate_mass" value="1.0"/>
+		<xacro:property name="top_plate_mass" value="0.1"/>
 		<!-- Wheels -->
-		<xacro:property name="wheel_radius" value="0.09"/>
+		<xacro:property name="wheel_radius" value="0.009"/>
 		<xacro:property name="wheel_thickness" value="0.04"/>
 		<xacro:property name="wheel_mass" value="0.1"/>
@@ -66,5 +66,5 @@
 				<material name="TopBlack"/>
 			</visual>
-			<xacro:inertial_box mass="1.0" x="${top_plate_length}" y="${top_plate_width}" z="${top_plate_height}">
+			<xacro:inertial_box mass="${top_plate_mass}" x="${top_plate_length}" y="${top_plate_width}" z="${top_plate_height}">
             	<origin xyz="0 0 ${top_plate_height/2}" rpy="0 0 0"/>
         	</xacro:inertial_box>
