Commit message: fixed couple of issues with the urdf

File: urdf/pioneer3dx/pioneer3dx.urdf.xacro (robot description, xacro)
@@ -33,4 +33,5 @@
 			<child link="${prefix}base_link"/>
 		</joint>
+		<!-- Top Plate -->
 		<link name="${prefix}top_plate">
 			<inertial>
@@ -57,4 +58,5 @@
 			<child link="${prefix}top_plate"/>
 		</joint>
+		<!-- Front Sonar -->
 		<link name="${prefix}front_sonar">
 			<inertial>
@@ -81,4 +83,5 @@
 			<child link="${prefix}front_sonar"/>
 		</joint>
+		<!-- Back Sonar -->
 		<joint name="${prefix}base_back_joint" type="fixed">
 			<origin xyz="0.109 0 0.209" rpy="0 0 0"/>
@@ -102,5 +105,5 @@
 			</visual>
 		</link>
-		<!-- Caster -->
+		<!-- Caster Swivel -->
 		<joint name="${prefix}base_caster_swivel_joint" type="continuous">
 			<origin xyz="-0.185 0 0.055" rpy="0 0 0"/>
@@ -155,4 +158,5 @@
 			<material value="Gazebo/Grey"/>
 		</gazebo>
+		<!-- Caster Wheel -->
 		<joint name="${prefix}caster_swivel_hubcap_joint" type="continuous">
 			<origin xyz="-0.026 0 -0.016" rpy="1.5708 0 0"/>
@@ -161,93 +165,95 @@
 			<child link="${prefix}caster_wheel"/>
 		</joint>
-			<link name="${prefix}caster_wheel">
-				<inertial>
-					<mass value="0.1"/>
-					<origin xyz="0 0 0"/>
-					<inertia ixx="0.012411765597" ixy="-0.000711733678" ixz="0.00050272983"
-										iyy="0.015218160428" iyz="-0.000004273467" izz="0.011763977943"/>
+		<link name="${prefix}caster_wheel">
+			<inertial>
+				<mass value="0.1"/>
+				<origin xyz="0 0 0"/>
+				<inertia ixx="0.012411765597" ixy="-0.000711733678" ixz="0.00050272983"
+						 iyy="0.015218160428" iyz="-0.000004273467" izz="0.011763977943"/>
 				</inertial>
-				<visual>
-					<origin xyz="0 0 0" rpy="0 0 0"/>
-					<geometry>
-						<cylinder radius="0.0375" length="0.01"/>
-					</geometry>
-					<material name="WheelBlack">
-						<color rgba="0.117 0.117 0.117 1"/>
-					</material>
-				</visual>
-				<collision>
-					<origin xyz="0 0 0" rpy="-1.5708 0 0"/>
-					<geometry>
-						<cylinder radius="0.0375" length="0.01"/>
-					</geometry>
-				</collision>
-			</link>
-			<joint name="${prefix}caster_wheel_joint" type="fixed">
-				<origin xyz="-0.0035 0 -0.001" rpy="1.5708 0 0"/>
-				<axis xyz="0 0 1"/>
-				<parent link="${prefix}caster_wheel"/>
-				<child link="${prefix}caster_hubcap"/>
-			</joint>
-			<link name="${prefix}left_hub">
-				<visual>
-					<origin xyz="0 0 0" rpy="${-3.1415927/2.0} 0 0"/>
-					<geometry>
-						<cylinder radius="0.09" length="0.01"/>
-					</geometry>
-					<material name="HubcapYellow">
-						<color rgba="1.0 0.811 0.151 1.0"/>
-					</material>
-				</visual>
-				<collision>
-					<origin xyz="0 0 0" rpy="${-3.1415927/2.0} 0 0"/>
-					<geometry>
-						<cylinder radius="0.09" length="0.01"/>
-					</geometry>
-				</collision>
-			</link>
-			<joint name="${prefix}left_hub_joint" type="fixed">
-				<origin xyz="0 0.15 0.08" rpy="0 0 0"/>
-				<parent link="${prefix}base_link"/>
-				<child link="${prefix}left_hub"/>
-				<axis xyz="0 1 0"/>
-			</joint>
-			<link name="${prefix}left_wheel">
-				<visual>
-					<origin xyz="0 0 0" rpy="1.5708 0 0"/>
-					<geometry>
-						<mesh filename="package://amr-ros-config/meshes/p3dx_meshes/left_wheel.stl"/>
-					</geometry>
-					<material name="WheelBlack">
-						<color rgba="0.117 0.117 0.117 1"/>
-					</material>
-				</visual>
-			</link>
-			<joint name="${prefix}left_wheel_joint" type="continuous">
+			<visual>
+				<origin xyz="0 0 0" rpy="0 0 0"/>
+				<geometry>
+					<cylinder radius="0.0375" length="0.01"/>
+				</geometry>
+				<material name="WheelBlack">
+					<color rgba="0.117 0.117 0.117 1"/>
+				</material>
+			</visual>
+			<collision>
 				<origin xyz="0 0 0" rpy="-1.5708 0 0"/>
-				<axis xyz="0 0 1"/>
-				<parent link="${prefix}left_hub"/>
-				<child link="${prefix}left_wheel"/>
-			</joint>
-			<gazebo reference="${prefix}left_wheel_joint">
-				<material value="Gazebo/Black"/>
-			</gazebo>
-			<link name="${prefix}right_hub">
-				<visual>
-					<origin xyz="0 0 0" rpy="${-3.1415927/2.0} 0 0"/>
-					<geometry>
-						<cylinder radius="0.09" length="0.01"/>
-					</geometry>
-					<material name="HubcapYellow">
-						<color rgba="1.0 0.811 0.151 1.0"/>
-					</material>
-				</visual>
-				<collision>
-					<origin xyz="0 0 0" rpy="${-3.1415927/2.0} 0 0"/>
-					<geometry>
-						<cylinder radius="0.09" length="0.01"/>
-					</geometry>
-				</collision>
-			</link>
+				<geometry>
+					<cylinder radius="0.0375" length="0.01"/>
+				</geometry>
+			</collision>
+		</link>
+		<joint name="${prefix}caster_wheel_joint" type="fixed">
+			<origin xyz="-0.0035 0 -0.001" rpy="1.5708 0 0"/>
+			<axis xyz="0 0 1"/>
+			<parent link="${prefix}caster_wheel"/>
+			<child link="${prefix}caster_hubcap"/>
+		</joint>
+		<!-- Left Wheel -->
+		<link name="${prefix}left_hub">
+			<visual>
+				<origin xyz="0 0 0" rpy="${-3.1415927/2.0} 0 0"/>
+				<geometry>
+					<cylinder radius="0.09" length="0.01"/>
+				</geometry>
+				<material name="HubcapYellow">
+					<color rgba="1.0 0.811 0.151 1.0"/>
+				</material>
+			</visual>
+			<collision>
+				<origin xyz="0 0 0" rpy="${-3.1415927/2.0} 0 0"/>
+				<geometry>
+					<cylinder radius="0.09" length="0.01"/>
+				</geometry>
+			</collision>
+		</link>
+		<joint name="${prefix}left_hub_joint" type="fixed">
+			<origin xyz="0 0.15 0.08" rpy="0 0 0"/>
+			<parent link="${prefix}base_link"/>
+			<child link="${prefix}left_hub"/>
+			<axis xyz="0 1 0"/>
+		</joint>
+		<link name="${prefix}left_wheel">
+			<visual>
+				<origin xyz="0 0 0" rpy="1.5708 0 0"/>
+				<geometry>
+					<mesh filename="package://amr-ros-config/meshes/p3dx_meshes/left_wheel.stl"/>
+				</geometry>
+				<material name="WheelBlack">
+					<color rgba="0.117 0.117 0.117 1"/>
+				</material>
+			</visual>
+		</link>
+		<joint name="${prefix}left_wheel_joint" type="continuous">
+			<origin xyz="0 0 0" rpy="-1.5708 0 0"/>
+			<axis xyz="0 0 1"/>
+			<parent link="${prefix}left_hub"/>
+			<child link="${prefix}left_wheel"/>
+		</joint>
+		<gazebo reference="${prefix}left_wheel_joint">
+			<material value="Gazebo/Black"/>
+		</gazebo>
+		<!-- Right Wheel -->
+		<link name="${prefix}right_hub">
+			<visual>
+				<origin xyz="0 0 0" rpy="${-3.1415927/2.0} 0 0"/>
+				<geometry>
+					<cylinder radius="0.09" length="0.01"/>
+				</geometry>
+				<material name="HubcapYellow">
+					<color rgba="1.0 0.811 0.151 1.0"/>
+				</material>
+			</visual>
+			<collision>
+				<origin xyz="0 0 0" rpy="${-3.1415927/2.0} 0 0"/>
+				<geometry>
+					<cylinder radius="0.09" length="0.01"/>
+				</geometry>
+			</collision>
+		</link>
 		<gazebo reference="${prefix}right_hub">
 			<material value="Gazebo/Yellow"/>
@@ -285,5 +291,5 @@
 				<leftJoint>${prefix}left_wheel_joint</leftJoint>
 				<rightJoint>${prefix}right_wheel_joint</rightJoint>
-				<wheelSeparation>0.158</wheelSeparation>
+				<wheelSeparation>0.3</wheelSeparation>
 				<wheelDiameter>0.12</wheelDiameter>
 				<torque>5</torque>

Commit message: flipped wheel direction

File: urdf/pioneer3dx/pioneer3dx.urdf.xacro (robot description, xacro)
@@ -105,4 +105,6 @@
 			<parent link="${prefix}base_link"/>
 			<child link="${prefix}caster_swivel"/>
+			<limit effort="10000.0" lower="-100000" upper="100000" velocity="100000"/>
+    		<dynamics damping="0.1" friction="0.1"/>
 		</joint>
 		<link name="${prefix}caster_swivel">
@@ -158,4 +160,6 @@
 			<parent link="${prefix}caster_swivel"/>
 			<child link="${prefix}caster_wheel"/>
+			<limit effort="10000.0" lower="-100000" upper="100000" velocity="100000"/>
+    		<dynamics damping="0.1" friction="0.1"/>
 		</joint>
 		<link name="${prefix}caster_wheel">
@@ -270,5 +274,5 @@
 		</link>
 		<joint name="${prefix}right_wheel_joint" type="continuous">
-			<origin xyz="0 0 0" rpy="1.5708 0 0"/>
+			<origin xyz="0 0 0" rpy="-1.5708 0 0"/>
 			<axis xyz="0 0 1"/>
 			<parent link="${prefix}right_hub"/>

Commit message: fixed passive joints

File: urdf/pioneer3dx/pioneer3dx.urdf.xacro (robot description, xacro)
@@ -100,5 +100,5 @@
 		</link>
 		<!-- Caster Swivel -->
-		<joint name="${prefix}base_caster_swivel_joint" type="continuous">
+		<joint name="${prefix}base_caster_swivel_joint" type="fixed"> <!--Not fixed. Change for simulation -->
 			<origin xyz="-0.185 0 0.055" rpy="0 0 0"/>
 			<axis xyz="0 0 1"/>
@@ -108,4 +108,5 @@
     		<dynamics damping="0.1" friction="0.1"/>
 		</joint>
+		<passive_joint name="${prefix}base_caster_swivel_joint"/> <!--Not working -->
 		<link name="${prefix}caster_swivel">
 			<inertial>
@@ -155,5 +156,5 @@
 		</gazebo>
 		<!-- Caster Wheel -->
-		<joint name="${prefix}caster_swivel_hubcap_joint" type="continuous">
+		<joint name="${prefix}caster_swivel_hubcap_joint" type="fixed"> <!--Not fixed. Change for simulation -->
 			<origin xyz="-0.026 0 -0.016" rpy="1.5708 0 0"/>
 			<axis xyz="0 0 1"/>
@@ -163,4 +164,5 @@
     		<dynamics damping="0.1" friction="0.1"/>
 		</joint>
+		<passive_joint name="${prefix}caster_swivel_hubcap_joint"/> <!--Not working -->
 		<link name="${prefix}caster_wheel">
 			<inertial>

Commit message: fixed simulation problems

File: urdf/pioneer3dx/pioneer3dx.urdf.xacro (robot description, xacro)
@@ -1,12 +1,14 @@
 <?xml version="1.0"?>
-<robot xmlns:xacro="http://ros.org/wiki/xacro">
+<robot xmlns:xacro="http://www.ros.org/wiki/xacro" >
 	<include filename="$(find amr-ros-config)/urdf/materials.xacro"/>
 	<xacro:macro name="pioneer3dx" params="prefix *origin">
 		<xacro:include filename="$(find amr-ros-config)/urdf/pioneer3dx/pioneer3dx_wheel.xacro"/>
+		<link name="${prefix}base_link">
+    	</link>
 		<!-- Base Link -->
-		<link name="${prefix}base_link">
+		<link name="${prefix}real_base_link">
 			<inertial>
 				<mass value="3.5"/>
-				<origin xyz="0 0 0"/>
+				<origin xyz="-0.045 0 0.148" rpy="0 0 0"/>
 				<inertia ixx="1" ixy="0" ixz="0" iyy="1" iyz="0" izz="1"/>
 			</inertial>
@@ -14,5 +16,5 @@
 				<origin xyz="-0.045 0 0.148" rpy="0 0 0"/>
 				<geometry>
-					<mesh filename="package://amr-ros-config/meshes/p3dx_meshes/chassis.stl"/>
+					<mesh filename="file://$(find amr-ros-config)/meshes/p3dx_meshes/chassis.stl"/>
 				</geometry>
 				<material name="ChassisRed">
@@ -21,10 +23,18 @@
 			</visual>
 			<collision>
-				<origin xyz="0 0 0" rpy="0 0 0"/>
-				<geometry>
-					<box size="0.01 0.01 0.01"/>
-				</geometry>
-			</collision>
-		</link>
+				<origin xyz="-0.045 0 0.148" rpy="0 0 0"/>
+				<geometry>
+					<mesh filename="file://$(find amr-ros-config)/meshes/p3dx_meshes/chassis.stl"/>
+				</geometry>
+			</collision>
+		</link>
+		<gazebo reference="${prefix}real_base_link">
+			<material>Gazebo/Red</material>
+		</gazebo>
+		<joint name="${prefix}real_base_link_joint" type="fixed">
+			<origin xyz="0 0 0" rpy="0 0 0"/>
+			<parent link="${prefix}base_link"/>
+			<child link="${prefix}real_base_link"/>
+		</joint>
 		<!-- Top Plate -->
 		<link name="${prefix}top_plate">
@@ -37,5 +47,5 @@
 				<origin xyz="0 0 0" rpy="0 0 0"/>
 				<geometry>
-					<mesh filename="package://amr-ros-config/meshes/p3dx_meshes/top.stl"/>
+					<mesh filename="file://$(find amr-ros-config)/meshes/p3dx_meshes/top.stl"/>
 				</geometry>
 				<material name="TopBlack">
@@ -43,4 +53,10 @@
 				</material>
 			</visual>
+			<collision>
+				<origin xyz="0 0 0" rpy="0 0 0"/>
+				<geometry>
+					<mesh filename="file://$(find amr-ros-config)/meshes/p3dx_meshes/top.stl"/>
+				</geometry>
+			</collision>
 		</link>
 		<gazebo reference="${prefix}top_plate">
@@ -49,5 +65,5 @@
 		<joint name="${prefix}base_top_joint" type="fixed">
 			<origin xyz="-0.045 0 0.234" rpy="0 0 0"/>
-			<parent link="${prefix}base_link"/>
+			<parent link="${prefix}real_base_link"/>
 			<child link="${prefix}top_plate"/>
 		</joint>
@@ -62,5 +78,5 @@
 				<origin xyz="0 0 0" rpy="0 0 0"/>
 				<geometry>
-					<mesh filename="package://amr-ros-config/meshes/p3dx_meshes/front_sonar.stl"/>
+					<mesh filename="file://$(find amr-ros-config)/meshes/p3dx_meshes/front_sonar.stl"/>
 				</geometry>
 				<material name="SonarYellow">
@@ -74,5 +90,5 @@
 		<joint name="${prefix}base_front_joint" type="fixed">
 			<origin xyz="-0.198 0 0.208" rpy="0 0 0"/>
-			<parent link="${prefix}base_link"/>
+			<parent link="${prefix}real_base_link"/>
 			<child link="${prefix}front_sonar"/>
 		</joint>
@@ -80,5 +96,5 @@
 		<joint name="${prefix}base_back_joint" type="fixed">
 			<origin xyz="0.109 0 0.209" rpy="0 0 0"/>
-			<parent link="${prefix}base_link"/>
+			<parent link="${prefix}real_base_link"/>
 			<child link="${prefix}back_sonar"/>
 		</joint>
@@ -92,5 +108,5 @@
 				<origin xyz="0 0 0" rpy="0 0 0"/>
 				<geometry>
-					<mesh filename="package://amr-ros-config/meshes/p3dx_meshes/back_sonar.stl"/>
+					<mesh filename="file://$(find amr-ros-config)/meshes/p3dx_meshes/back_sonar.stl"/>
 				</geometry>
 				<material name="SonarYellow">
@@ -103,8 +119,8 @@
 			<origin xyz="-0.185 0 0.055" rpy="0 0 0"/>
 			<axis xyz="0 0 1"/>
-			<parent link="${prefix}base_link"/>
+			<parent link="${prefix}real_base_link"/>
 			<child link="${prefix}caster_swivel"/>
 			<limit effort="10000.0" lower="-100000" upper="100000" velocity="100000"/>
-    		<dynamics damping="0.1" friction="0.1"/>
+    		<dynamics damping="0.001" friction="0.0001"/>
 		</joint>
 		<passive_joint name="${prefix}base_caster_swivel_joint"/> <!--Not working -->
@@ -118,5 +134,5 @@
 				<origin xyz="0 0 0" rpy="0 0 0"/>
 				<geometry>
-					<mesh filename="package://amr-ros-config/meshes/p3dx_meshes/caster_swivel.stl"/>
+					<mesh filename="file://$(find amr-ros-config)/meshes/p3dx_meshes/caster_swivel.stl"/>
 				</geometry>
 				<material name="caster_swivel">
@@ -124,4 +140,10 @@
 				</material>
 			</visual>
+			<collision>
+				<origin xyz="0 0 0" rpy="0 0 0"/>
+				<geometry>
+					<mesh filename="file://$(find amr-ros-config)/meshes/p3dx_meshes/caster_swivel.stl"/>
+				</geometry>
+			</collision>
 		</link>
 		<gazebo reference="${prefix}caster_swivel">
@@ -134,10 +156,10 @@
 				<origin xyz="0 0 0"/>
 				<inertia ixx="0.012411765597" ixy="-0.000711733678" ixz="0.00050272983"
-								 iyy="0.015218160428" iyz="-0.000004273467" izz="0.011763977943"/>
-			</inertial>
-			<visual>
-				<origin xyz="0 0 0" rpy="0 0 0"/>
-				<geometry>
-					<mesh filename="package://amr-ros-config/meshes/p3dx_meshes/caster_hubcap.stl"/>
+							iyy="0.015218160428" iyz="-0.000004273467" izz="0.011763977943"/>
+			</inertial>
+			<visual>
+				<origin xyz="0 0 0" rpy="0 0 0"/>
+				<geometry>
+					<mesh filename="file://$(find amr-ros-config)/meshes/p3dx_meshes/caster_hubcap.stl"/>
 				</geometry>
 				<material name="caster_swivel">
@@ -148,5 +170,5 @@
 				<origin xyz="0 0 0" rpy="0 0 0"/>
 				<geometry>
-					<box size="0.05 0.05 0.05"/>
+					<mesh filename="file://$(find amr-ros-config)/meshes/p3dx_meshes/caster_hubcap.stl"/>
 				</geometry>
 			</collision>
@@ -162,5 +184,5 @@
 			<child link="${prefix}caster_wheel"/>
 			<limit effort="10000.0" lower="-100000" upper="100000" velocity="100000"/>
-    		<dynamics damping="0.1" friction="0.1"/>
+    		<dynamics damping="0.001" friction="0.0001"/>
 		</joint>
 		<passive_joint name="${prefix}caster_swivel_hubcap_joint"/> <!--Not working -->
@@ -171,5 +193,5 @@
 				<inertia ixx="0.012411765597" ixy="-0.000711733678" ixz="0.00050272983"
 						 iyy="0.015218160428" iyz="-0.000004273467" izz="0.011763977943"/>
-				</inertial>
+			</inertial>
 			<visual>
 				<origin xyz="0 0 0" rpy="0 0 0"/>
@@ -182,5 +204,5 @@
 			</visual>
 			<collision>
-				<origin xyz="0 0 0" rpy="-1.5708 0 0"/>
+				<origin xyz="0 0 0" rpy="0 0 0"/>
 				<geometry>
 					<cylinder radius="0.0375" length="0.01"/>
@@ -188,4 +210,7 @@
 			</collision>
 		</link>
+		<gazebo reference="${prefix}caster_hubcap">
+			<material value="Gazebo/Grey"/>
+		</gazebo>
 		<joint name="${prefix}caster_wheel_joint" type="fixed">
 			<origin xyz="-0.0035 0 -0.001" rpy="1.5708 0 0"/>
@@ -211,8 +236,13 @@
 				</geometry>
 			</collision>
+			<inertial>
+				<mass value="0.1"/>
+				<origin xyz="0 0 0"/>
+				<inertia ixx="0.001" ixy="0" ixz="0" iyy="0.001" iyz="0" izz="0.001"/>
+			</inertial>
 		</link>
 		<joint name="${prefix}left_hub_joint" type="fixed">
 			<origin xyz="0 0.15 0.08" rpy="0 0 0"/>
-			<parent link="${prefix}base_link"/>
+			<parent link="${prefix}real_base_link"/>
 			<child link="${prefix}left_hub"/>
 			<axis xyz="0 1 0"/>
@@ -222,5 +252,5 @@
 				<origin xyz="0 0 0" rpy="1.5708 0 0"/>
 				<geometry>
-					<mesh filename="package://amr-ros-config/meshes/p3dx_meshes/left_wheel.stl"/>
+					<mesh filename="file://$(find amr-ros-config)/meshes/p3dx_meshes/left_wheel.stl"/>
 				</geometry>
 				<material name="WheelBlack">
@@ -228,5 +258,19 @@
 				</material>
 			</visual>
-		</link>
+			<collision>
+				<origin xyz="0 0 0" rpy="1.5708 0 0"/>
+				<geometry>
+					<mesh filename="file://$(find amr-ros-config)/meshes/p3dx_meshes/left_wheel.stl"/>
+				</geometry>
+			</collision>
+			<inertial>
+				<mass value="0.5"/>
+				<origin xyz="0 0 0"/>
+				<inertia ixx="0.001" ixy="0" ixz="0" iyy="0.001" iyz="0" izz="0.001"/>
+			</inertial>
+		</link>
+		<gazebo reference="${prefix}left_wheel">
+			<material value="Gazebo/Black"/>
+		</gazebo>
 		<joint name="${prefix}left_wheel_joint" type="continuous">
 			<origin xyz="0 0 0" rpy="-1.5708 0 0"/>
@@ -234,8 +278,6 @@
 			<parent link="${prefix}left_hub"/>
 			<child link="${prefix}left_wheel"/>
-		</joint>
-		<gazebo reference="${prefix}left_wheel_joint">
-			<material value="Gazebo/Black"/>
-		</gazebo>
+			<dynamics damping="0.001" friction="0.0001"/>
+		</joint>
 		<!-- Right Wheel -->
 		<link name="${prefix}right_hub">
@@ -252,7 +294,12 @@
 				<origin xyz="0 0 0" rpy="${-3.1415927/2.0} 0 0"/>
 				<geometry>
-					<cylinder radius="0.09" length="0.01"/>
-				</geometry>
-			</collision>
+					<cylinder radius="0.06" length="0.04"/>
+				</geometry>
+			</collision>
+			<inertial>
+				<mass value="0.1"/>
+				<origin xyz="0 0 0"/>
+				<inertia ixx="0.001" ixy="0" ixz="0" iyy="0.001" iyz="0" izz="0.001"/>
+			</inertial>
 		</link>
 		<gazebo reference="${prefix}right_hub">
@@ -261,5 +308,5 @@
 		<joint name="${prefix}right_hub_joint" type="fixed">
 			<origin xyz="0 -0.15 0.08" rpy="0 0 0"/>
-			<parent link="${prefix}base_link"/>
+			<parent link="${prefix}real_base_link"/>
 			<child link="${prefix}right_hub"/>
 		</joint>
@@ -268,5 +315,5 @@
 				<origin xyz="0 0 0" rpy="-1.5708 0 0"/>
 				<geometry>
-					<mesh filename="package://amr-ros-config/meshes/p3dx_meshes/right_wheel.stl"/>
+					<mesh filename="file://$(find amr-ros-config)/meshes/p3dx_meshes/right_wheel.stl"/>
 				</geometry>
 				<material name="WheelBlack">
@@ -274,5 +321,19 @@
 				</material>
 			</visual>
-		</link>
+			<collision>
+				<origin xyz="0 0 0" rpy="-1.5708 0 0"/>
+				<geometry>
+					<mesh filename="file://$(find amr-ros-config)/meshes/p3dx_meshes/right_wheel.stl"/>
+				</geometry>
+			</collision>
+			<inertial>
+				<mass value="0.5"/>
+				<origin xyz="0 0 0"/>
+				<inertia ixx="0.001" ixy="0" ixz="0" iyy="0.001" iyz="0" izz="0.001"/>
+			</inertial>
+		</link>
+		<gazebo reference="${prefix}right_wheel">
+			<material value="Gazebo/Black"/>
+		</gazebo>
 		<joint name="${prefix}right_wheel_joint" type="continuous">
 			<origin xyz="0 0 0" rpy="-1.5708 0 0"/>
@@ -280,24 +341,23 @@
 			<parent link="${prefix}right_hub"/>
 			<child link="${prefix}right_wheel"/>
-		</joint>
-		<gazebo reference="${prefix}right_wheel_joint">
-			<material value="Gazebo/Black"/>
-		</gazebo>
+			<dynamics damping="0.001" friction="0.0001"/>
+		</joint>
 		<!-- Gazebo plugin -->
-		<gazebo>
-			<plugin name="differential_drive_controller" filename="libgazebo_ros_diff_drive.so">
-				<alwaysOn>true</alwaysOn>
-				<updateRate>100</updateRate>
-				<leftJoint>${prefix}left_wheel_joint</leftJoint>
-				<rightJoint>${prefix}right_wheel_joint</rightJoint>
-				<wheelSeparation>0.3</wheelSeparation>
-				<wheelDiameter>0.12</wheelDiameter>
-				<torque>5</torque>
-				<commandTopic>cmd_vel</commandTopic>
-				<robotBaseFrame>${prefix}base_link</robotBaseFrame>
-				<odometryTopic>odom</odometryTopic>
-				<odometryFrame>odom</odometryFrame>
+		<!-- <gazebo>
+			<plugin name="diff_drive" filename="libgazebo_ros_diff_drive.so">
+				<left_joint>${prefix}left_wheel_joint</left_joint>
+				<right_joint>${prefix}right_wheel_joint</right_joint>
+				<wheel_separation>0.3</wheel_separation>
+				<wheel_diameter>0.12</wheel_diameter>
+				<max_wheel_torque>200</max_wheel_torque>
+				<max_wheel_acceleration>10.0</max_wheel_acceleration>
+				<command_topic>cmd_vel</command_topic>
+				<robot_base_frame>${prefix}real_base_link</robot_base_frame>
+				<odometry_frame>${prefix}odom</odometry_frame>
+				<publish_odom>true</publish_odom>
+				<publish_odom_tf>true</publish_odom_tf>
+				<publish_wheel_tf>true</publish_wheel_tf>
 			</plugin>
-		</gazebo>
+		</gazebo> -->
 	</xacro:macro>
 </robot>
