Commit message: new simulation attempt

File: urdf/pioneer3dx/gazebo_control.xacro (robot description, xacro)
@@ -3,10 +3,32 @@
     <xacro:macro name="pioneer3dx_gazebo_control" params="prefix">
         <gazebo>
+            <plugin
+                filename="gz-sim-diff-drive-system"
+                name="gz::sim::systems::DiffDrive">
+                <left_joint>${prefix}left_wheel_joint</left_joint>
+                <right_joint>${prefix}right_wheel_joint</right_joint>
+                <wheel_separation>0.1</wheel_separation>
+                <wheel_radius>0.03</wheel_radius>
+                <odom_publish_frequency>1</odom_publish_frequency>
+                <topic>cmd_vel</topic>
+            </plugin>
+            <plugin
+                filename="gz-sim-joint-state-publisher-system"
+                name="gz::sim::systems::JointStatePublisher">
+            </plugin>
+            <plugin
+                filename="ignition-gazebo-pose-publisher-system"
+                name="ignition::gazebo::systems::PosePublisher">
+                <publish_link_pose>true</publish_link_pose>
+                <use_pose_vector_msg>true</use_pose_vector_msg>
+            </plugin>
+        </gazebo>
+        <!-- <gazebo>
             <plugin name="gazebo_ros2_control" filename="libgazebo_ros2_control.so">
                 <parameters>$(find amr-ros-config)/config/controller_config.yaml</parameters>
 				<parameters>$(find amr-ros-config)/config/gazebo_params.yaml</parameters>
             </plugin>
-        </gazebo>
-        <ros2_control name="GazeboSystem" type="system">
+        </gazebo> -->
+        <!-- <ros2_control name="GazeboSystem" type="system">
             <hardware>
                 <plugin>gazebo_ros2_control/GazeboSystem</plugin>
@@ -28,5 +50,5 @@
                 <state_interface name="position"/>
             </joint>
-        </ros2_control>
+        </ros2_control> -->
     </xacro:macro>
 </robot>

File: urdf/pioneer3dx/pioneer3dx_sim.urdf.xacro (robot description, xacro)
@@ -12,6 +12,6 @@
 		<xacro:property name="chassis_height" value="0.172"/>
 		<link name="${prefix}real_base_link">
-			<xacro:inertial_box mass="7.0" x="${chassis_length}" y="${chassis_width}" z="${chassis_height}">
-            	<origin xyz="${-chassis_length/2} 0 ${chassis_height/2}" rpy="0 0 0"/>
+			<xacro:inertial_box mass="3.5" x="${-chassis_length}" y="${chassis_width}" z="${chassis_height}">
+            	<origin xyz="0 0 0" rpy="0 0 0"/>
         	</xacro:inertial_box>
 			<visual>
@@ -42,5 +42,5 @@
 		<xacro:property name="top_plate_height" value="0.0052"/>
 		<link name="${prefix}top_plate">
-			<xacro:inertial_box mass="0.1" x="${top_plate_length}" y="${top_plate_width}" z="${top_plate_height}">
+			<xacro:inertial_box mass="0.001" x="${top_plate_length}" y="${top_plate_width}" z="${top_plate_height}">
             	<origin xyz="${chassis_length/2} 0 ${chassis_height/2}" rpy="0 0 0"/>
         	</xacro:inertial_box>
@@ -114,5 +114,5 @@
 		</gazebo>
 		<!-- Caster Swivel -->
-		<joint name="${prefix}base_caster_swivel_joint" type="continuous"> <!--Not fixed. Change for simulation -->
+		<joint name="${prefix}base_caster_swivel_joint" type="fixed"> <!--Not fixed. Change for simulation -->
 			<origin xyz="-0.185 0 0.055" rpy="0 0 0"/>
 			<axis xyz="0 0 1"/>
@@ -181,5 +181,5 @@
 		<!-- Caster Wheel -->
 		<link name="${prefix}caster_wheel">
-			<xacro:inertial_cylinder mass="0.2" length="0.01" radius="0.0375">
+			<xacro:inertial_cylinder mass="2.0" length="0.01" radius="0.0375">
 				<origin xyz="0 0 0" rpy="0 0 0"/>
 			</xacro:inertial_cylinder>
@@ -201,6 +201,8 @@
 		<gazebo reference="${prefix}caster_wheel">
 			<material value="Gazebo/Black"/>
-		</gazebo>
-		<joint name="${prefix}caster_wheel_joint" type="continuous">  <!--Not fixed. Change for simulation -->
+			<mu1 value="0.0001"/>
+        	<mu2 value="0.0001"/>
+		</gazebo>
+		<joint name="${prefix}caster_wheel_joint" type="fixed">  <!--Not fixed. Change for simulation -->
 			<origin xyz="-0.0035 0 -0.001" rpy="0 0 0"/>
 			<axis xyz="0 0 1"/>
@@ -224,5 +226,5 @@
 			</collision> -->
 			<inertial>
-				<mass value="0.1"/>
+				<mass value="0.01"/>
 				<origin xyz="0 0 0" rpy="${-3.1415927/2.0} 0 0"/>
 				<inertia ixx="0.001" ixy="0" ixz="0" iyy="0.001" iyz="0" izz="0.001"/>
@@ -249,8 +251,8 @@
 				<origin xyz="0 0 0" rpy="0 0 0"/>
 				<geometry>
-					<cylinder radius="0.09" length="0.04"/>
+					<sphere radius="0.09"/>
 				</geometry>
 			</collision>
-			<xacro:inertial_cylinder mass="2.0" length="0.04" radius="0.09">
+			<xacro:inertial_cylinder mass="0.5" length="0.04" radius="0.09">
 				<origin xyz="0 0 0" rpy="0 0 0"/>
 			</xacro:inertial_cylinder>
@@ -259,4 +261,6 @@
 		<gazebo reference="${prefix}left_wheel">
 			<material value="Gazebo/Black"/>
+			<mu1 value="0.9"/>
+        	<mu2 value="0.9"/>
 		</gazebo>
 		<joint name="${prefix}left_wheel_joint" type="continuous">
@@ -283,5 +287,5 @@
 			</collision> -->
 			<inertial>
-				<mass value="0.1"/>
+				<mass value="0.01"/>
 				<origin xyz="0 0 0" rpy="${3.1415927/2.0} 0 0"/>
 				<inertia ixx="0.001" ixy="0" ixz="0" iyy="0.001" iyz="0" izz="0.001"/>
@@ -307,8 +311,8 @@
 				<origin xyz="0 0 0" rpy="0 0 0"/>
 				<geometry>
-					<cylinder radius="0.09" length="0.04"/>
+					<sphere radius="0.09"/>
 				</geometry>
 			</collision>
-			<xacro:inertial_cylinder mass="2.0" length="0.04" radius="0.09">
+			<xacro:inertial_cylinder mass="0.5" length="0.04" radius="0.09">
 				<origin xyz="0 0 0" rpy="0 0 0"/>
 			</xacro:inertial_cylinder>
@@ -317,4 +321,6 @@
 		<gazebo reference="${prefix}right_wheel">
 			<material value="Gazebo/Black"/>
+			<mu1 value="0.9"/>
+        	<mu2 value="0.9"/>
 		</gazebo>
 		<joint name="${prefix}right_wheel_joint" type="continuous">

Commit message: fix diff drive, 1st attempt

File: urdf/pioneer3dx/gazebo_control.xacro (robot description, xacro)
@@ -3,21 +3,19 @@
     <xacro:macro name="pioneer3dx_gazebo_control" params="prefix">
         <gazebo>
-            <plugin name="gazebo_ros2_control" filename="libgazebo_ros2_control.so">
-                <parameters>$(find amr-ros-config)/config/controller_config.yaml</parameters>
-				<parameters>$(find amr-ros-config)/config/gazebo_params.yaml</parameters>
-            </plugin>
-            <plugin name="gazebo_ros_p3d" filename="libgazebo_ros_p3d.so">
-                <ros>
-                    <!-- Use your desired namespace or leave empty for default -->
-                    <namespace>/galax_robot</namespace>
-                    <!-- The topic name where the position will be published -->
-                    <remapping>odom:=/galax_pose</remapping>
-                </ros>
-                <!-- Replace with your robot's main link -->
-                <body_name>pioneer3dx_base_link</body_name>
-                <!-- Update rate in Hz -->
-                <update_rate>30.0</update_rate>
-                <xyzOffsets>0 0 0</xyzOffsets>
-                <rpyOffsets>0 0 0</rpyOffsets>
+            <plugin name="diff_drive" filename="libgazebo_ros_diff_drive.so">
+                <!-- Wheel Information -->
+                <left_joint>${prefix}left_wheel_joint</left_joint>
+                <right_joint>${prefix}right_wheel_joint</right_joint>
+                <wheel_separation>0.30</wheel_separation>
+                <wheel_diameter>0.18</wheel_diameter>
+                <!-- Limits -->
+                <max_wheel_torque>200</max_wheel_torque>
+                <max_wheel_acceleration>10.0</max_wheel_acceleration>
+                <!-- Output -->
+                <odometry_frame>${prefix}odom</odometry_frame>
+                <robot_base_frame>${prefix}base_link</robot_base_frame>
+                <publish_odom>true</publish_odom>
+                <publish_odom_tf>true</publish_odom_tf>
+                <publish_wheel_tf>true</publish_wheel_tf>
             </plugin>
         </gazebo>
@@ -43,4 +41,10 @@
             </joint>
         </ros2_control>
+        <gazebo>
+            <plugin name="gazebo_ros2_control" filename="libgazebo_ros2_control.so">
+                <parameters>$(find amr-ros-config)/config/controller_config.yaml</parameters>
+				<parameters>$(find amr-ros-config)/config/gaz_ros2_ctl_use_sim.yaml</parameters>
+            </plugin>
+        </gazebo>
     </xacro:macro>
 </robot>

File: urdf/pioneer3dx/pioneer3dx_sim.urdf.xacro (robot description, xacro)
@@ -15,4 +15,5 @@
 		<xacro:property name="top_plate_width" value="0.272"/>
 		<xacro:property name="top_plate_height" value="0.0052"/>
+		<xacro:property name="top_plate_mass" value="1.0"/>
 		<!-- Wheels -->
 		<xacro:property name="wheel_radius" value="0.09"/>
@@ -25,10 +26,10 @@
 		<!-- Chasis -->
 		<link name="${prefix}real_base_link">
-			<collision>
+			<!-- <collision>
 				<origin xyz="${chassis_length/2} 0 ${chassis_height/2}"/>
 				<geometry>
 					<box size="${chassis_length} ${chassis_width} ${chassis_height}"/>
 				</geometry>
-			</collision>
+			</collision> -->
 			<visual>
 				<origin xyz="-0.045 0 0.148" rpy="0 0 0"/>
@@ -39,5 +40,5 @@
 			</visual>
 			<xacro:inertial_box mass="${chassis_mass}" x="${chassis_length}" y="${chassis_width}" z="${chassis_height}">
-            	<origin xyz="${-chassis_length/2} 0 ${chassis_height/2}" rpy="0 0 0"/>
+            	<origin xyz="${-chassis_length/2} 0 ${-chassis_height/2}" rpy="0 0 0"/>
         	</xacro:inertial_box>
 		</link>
@@ -52,10 +53,10 @@
 		<!-- Top Plate -->
 		<link name="${prefix}top_plate">
-			<collision>
+			<!-- <collision>
 				<origin xyz="${top_plate_length/2} 0 ${top_plate_height/2}"/>
 				<geometry>
 					<box size="${top_plate_length} ${top_plate_width} ${top_plate_height}"/>
 				</geometry>
-			</collision>
+			</collision> -->
 			<visual>
 				<origin xyz="0 0 0" rpy="0 0 0"/>
@@ -147,5 +148,5 @@
 			<material value="Gazebo/Grey"/>
 		</gazebo>
-		<joint name="${prefix}base_caster_swivel_joint" type="continuous"> <!--Not fixed. Change for simulation -->
+		<joint name="${prefix}base_caster_swivel_joint" type="fixed"> <!--Not fixed. Change for simulation -->
 			<origin xyz="-0.185 0 0.055" rpy="0 0 0"/>
 			<axis xyz="0 0 1"/>
