Commit message: simulation fixed. Still drifting

File: urdf/pioneer3dx/pioneer3dx_sim.urdf.xacro (robot description, xacro)
@@ -114,5 +114,5 @@
 		</gazebo>
 		<!-- Caster Swivel -->
-		<joint name="${prefix}base_caster_swivel_joint" type="fixed"> <!--Not fixed. Change for simulation -->
+		<joint name="${prefix}base_caster_swivel_joint" type="continuous"> <!--Not fixed. Change for simulation -->
 			<origin xyz="-0.185 0 0.055" rpy="0 0 0"/>
 			<axis xyz="0 0 1"/>
@@ -202,5 +202,5 @@
 			<material value="Gazebo/Black"/>
 		</gazebo>
-		<joint name="${prefix}caster_wheel_joint" type="fixed">  <!--Not fixed. Change for simulation -->
+		<joint name="${prefix}caster_wheel_joint" type="continuous">  <!--Not fixed. Change for simulation -->
 			<origin xyz="-0.0035 0 -0.001" rpy="0 0 0"/>
 			<axis xyz="0 0 1"/>

Commit message: fixed drifting

File: urdf/pioneer3dx/pioneer3dx_sim.urdf.xacro (robot description, xacro)
@@ -4,5 +4,4 @@
 	<xacro:include filename="$(find amr-ros-config)/urdf/inertial_macros.xacro"/>
 	<xacro:macro name="pioneer3dx" params="prefix *origin">
-		<!-- <xacro:include filename="$(find amr-ros-config)/urdf/pioneer3dx/pioneer3dx_wheel.xacro"/> -->
 		<link name="${prefix}base_link">
     	</link>
@@ -12,5 +11,5 @@
 		<xacro:property name="chassis_height" value="0.172"/>
 		<link name="${prefix}real_base_link">
-			<xacro:inertial_box mass="7.0" x="${chassis_length}" y="${chassis_width}" z="${chassis_height}">
+			<xacro:inertial_box mass="30.0" x="${chassis_length}" y="${chassis_width}" z="${chassis_height}">
             	<origin xyz="${-chassis_length/2} 0 ${chassis_height/2}" rpy="0 0 0"/>
         	</xacro:inertial_box>
@@ -22,10 +21,4 @@
 				<material name="ChassisRed"/>
 			</visual>
-			<!-- <collision>
-				<origin xyz="-0.045 0 0.148" rpy="0 0 0"/>
-				<geometry>
-					<mesh filename="file://$(find amr-ros-config)/meshes/p3dx_meshes/chassis.stl"/>
-				</geometry>
-			</collision> -->
 		</link>
 		<gazebo reference="${prefix}real_base_link">
@@ -42,6 +35,6 @@
 		<xacro:property name="top_plate_height" value="0.0052"/>
 		<link name="${prefix}top_plate">
-			<xacro:inertial_box mass="0.1" x="${top_plate_length}" y="${top_plate_width}" z="${top_plate_height}">
-            	<origin xyz="${chassis_length/2} 0 ${chassis_height/2}" rpy="0 0 0"/>
+			<xacro:inertial_box mass="1.0" x="${top_plate_length}" y="${top_plate_width}" z="${top_plate_height}">
+            	<origin xyz="0 0 ${top_plate_height/2}" rpy="0 0 0"/>
         	</xacro:inertial_box>
 			<visual>
@@ -125,5 +118,5 @@
 		<link name="${prefix}caster_swivel">
 			<inertial>
-				<mass value="0.01"/>
+				<mass value="0.1"/>
 				<origin xyz="0 0 0"/>
 				<inertia ixx="0.01" ixy="0" ixz="0" iyy="0.01" iyz="0" izz="0.01"/>
@@ -149,5 +142,5 @@
 		<link name="${prefix}caster_hubcap">
 			<inertial>
-				<mass value="0.01"/>
+				<mass value="0.1"/>
 				<origin xyz="0 0 0"/>
 				<inertia ixx="0.012411765597" ixy="-0.000711733678" ixz="0.00050272983"
@@ -181,5 +174,5 @@
 		<!-- Caster Wheel -->
 		<link name="${prefix}caster_wheel">
-			<xacro:inertial_cylinder mass="0.2" length="0.01" radius="0.0375">
+			<xacro:inertial_cylinder mass="2.0" length="0.01" radius="0.0375">
 				<origin xyz="0 0 0" rpy="0 0 0"/>
 			</xacro:inertial_cylinder>
@@ -200,7 +193,14 @@
 		</link>
 		<gazebo reference="${prefix}caster_wheel">
-			<material value="Gazebo/Black"/>
-		</gazebo>
-		<joint name="${prefix}caster_wheel_joint" type="continuous">  <!--Not fixed. Change for simulation -->
+			<material value="Gazebo/White"/>
+			<kp>1000000.0</kp> <!-- kp and kd for rubber -->
+			<kd>100.0</kd>
+			<mu1>0.0</mu1>
+			<mu2>0.0</mu2>
+			<!-- fdir1 0 1 0 /fdir1 --> <!-- see http://github.com/MobileRobots/amr-ros-config/issues/6 -->
+			<maxVel>1.0</maxVel>
+			<minDepth>0.00</minDepth>
+		</gazebo>
+		<joint name="${prefix}caster_wheel_joint" type="fixed">  <!--Not fixed. Change for simulation -->
 			<origin xyz="-0.0035 0 -0.001" rpy="0 0 0"/>
 			<axis xyz="0 0 1"/>
@@ -249,8 +249,8 @@
 				<origin xyz="0 0 0" rpy="0 0 0"/>
 				<geometry>
-					<cylinder radius="0.09" length="0.04"/>
+					<sphere radius="0.09"/>
 				</geometry>
 			</collision>
-			<xacro:inertial_cylinder mass="2.0" length="0.04" radius="0.09">
+			<xacro:inertial_cylinder mass="20.0" length="0.04" radius="0.09">
 				<origin xyz="0 0 0" rpy="0 0 0"/>
 			</xacro:inertial_cylinder>
@@ -259,4 +259,11 @@
 		<gazebo reference="${prefix}left_wheel">
 			<material value="Gazebo/Black"/>
+			<kp>1000000.0</kp> <!-- kp and kd for rubber -->
+			<kd>100.0</kd>
+			<mu1>1.0</mu1>
+			<mu2>1.0</mu2>
+			<!-- fdir1 0 1 0 /fdir1 --> <!-- see http://github.com/MobileRobots/amr-ros-config/issues/6 -->
+			<maxVel>1.0</maxVel>
+			<minDepth>0.00</minDepth>
 		</gazebo>
 		<joint name="${prefix}left_wheel_joint" type="continuous">
@@ -276,10 +283,4 @@
 				<material name="HubcapYellow"/>
 			</visual>
-			<!-- <collision>
-				<origin xyz="0 0 0" rpy="${-3.1415927/2.0} 0 0"/>
-				<geometry>
-					<cylinder radius="0.06" length="0.04"/>
-				</geometry>
-			</collision> -->
 			<inertial>
 				<mass value="0.1"/>
@@ -307,8 +308,8 @@
 				<origin xyz="0 0 0" rpy="0 0 0"/>
 				<geometry>
-					<cylinder radius="0.09" length="0.04"/>
+					<sphere radius="0.09"/>
 				</geometry>
 			</collision>
-			<xacro:inertial_cylinder mass="2.0" length="0.04" radius="0.09">
+			<xacro:inertial_cylinder mass="20.0" length="0.04" radius="0.09">
 				<origin xyz="0 0 0" rpy="0 0 0"/>
 			</xacro:inertial_cylinder>
@@ -317,4 +318,11 @@
 		<gazebo reference="${prefix}right_wheel">
 			<material value="Gazebo/Black"/>
+			<kp>1000000.0</kp> <!-- kp and kd for rubber -->
+			<kd>100.0</kd>
+			<mu1>1.0</mu1>
+			<mu2>1.0</mu2>
+			<!-- fdir1 0 1 0 /fdir1 --> <!-- see http://github.com/MobileRobots/amr-ros-config/issues/6 -->
+			<maxVel>1.0</maxVel>
+			<minDepth>0.01</minDepth>
 		</gazebo>
 		<joint name="${prefix}right_wheel_joint" type="continuous">
@@ -325,19 +333,10 @@
 			<dynamics damping="0.001" friction="0.0001"/>
 		</joint>
-		<!-- Gazebo plugin -->
 		<!-- <gazebo>
-			<plugin name="diff_drive" filename="libgazebo_ros_diff_drive.so">
-				<left_joint>${prefix}left_wheel_joint</left_joint>
-				<right_joint>${prefix}right_wheel_joint</right_joint>
-				<wheel_separation>0.3</wheel_separation>
-				<wheel_diameter>0.12</wheel_diameter>
-				<max_wheel_torque>200</max_wheel_torque>
-				<max_wheel_acceleration>10.0</max_wheel_acceleration>
-				<command_topic>cmd_vel</command_topic>
-				<robot_base_frame>${prefix}real_base_link</robot_base_frame>
-				<odometry_frame>${prefix}odom</odometry_frame>
-				<publish_odom>true</publish_odom>
-				<publish_odom_tf>true</publish_odom_tf>
-				<publish_wheel_tf>true</publish_wheel_tf>
+			<plugin name="ground_plane" filename="libgazebo_ros_surface_properties.so">
+				<mu>1.0</mu>
+				<mu2>1.0</mu2>
+				<kp>100000</kp>
+				<kd>1</kd>
 			</plugin>
 		</gazebo> -->

Commit message: changes in dynamics

File: urdf/pioneer3dx/pioneer3dx_sim.urdf.xacro (robot description, xacro)
@@ -190,5 +190,5 @@
 				</geometry>
 			</collision>
-			<dynamics damping="10.0" friction="0"/>
+			<dynamics damping="0.0001" friction="0.0001"/>
 		</link>
 		<gazebo reference="${prefix}caster_wheel">
@@ -207,4 +207,5 @@
 			<parent link="${prefix}caster_hubcap"/>
 			<child link="${prefix}caster_wheel"/>
+			<dynamics damping="1.0" friction="1.0"/>
 		</joint>
 		<!-- Left Wheel -->
@@ -252,8 +253,8 @@
 				</geometry>
 			</collision>
-			<xacro:inertial_cylinder mass="20.0" length="0.04" radius="0.09">
+			<xacro:inertial_cylinder mass="2.0" length="0.04" radius="0.09">
 				<origin xyz="0 0 0" rpy="0 0 0"/>
 			</xacro:inertial_cylinder>
-			<dynamics damping="0" friction="10.0"/>
+			<dynamics damping="1.0" friction="1.0"/>
 		</link>
 		<gazebo reference="${prefix}left_wheel">
@@ -272,5 +273,5 @@
 			<parent link="${prefix}left_hub"/>
 			<child link="${prefix}left_wheel"/>
-			<dynamics damping="0.001" friction="0.0001"/>
+			<dynamics damping="1.0" friction="1.0"/>
 		</joint>
 		<!-- Right Wheel -->
@@ -311,8 +312,8 @@
 				</geometry>
 			</collision>
-			<xacro:inertial_cylinder mass="20.0" length="0.04" radius="0.09">
+			<xacro:inertial_cylinder mass="2.0" length="0.04" radius="0.09">
 				<origin xyz="0 0 0" rpy="0 0 0"/>
 			</xacro:inertial_cylinder>
-			<dynamics damping="0" friction="10.0"/>
+			<!-- <dynamics damping="1.0" friction="1.0"/> -->
 		</link>
 		<gazebo reference="${prefix}right_wheel">
@@ -331,5 +332,5 @@
 			<parent link="${prefix}right_hub"/>
 			<child link="${prefix}right_wheel"/>
-			<dynamics damping="0.001" friction="0.0001"/>
+			<dynamics damping="1.0" friction="1.0"/>
 		</joint>
 		<!-- <gazebo>

Commit message: polished

File: urdf/pioneer3dx/pioneer3dx_sim.urdf.xacro (robot description, xacro)
@@ -253,5 +253,5 @@
 				</geometry>
 			</collision>
-			<xacro:inertial_cylinder mass="2.0" length="0.04" radius="0.09">
+			<xacro:inertial_cylinder mass="20.0" length="0.04" radius="0.09">
 				<origin xyz="0 0 0" rpy="0 0 0"/>
 			</xacro:inertial_cylinder>
@@ -273,5 +273,5 @@
 			<parent link="${prefix}left_hub"/>
 			<child link="${prefix}left_wheel"/>
-			<dynamics damping="1.0" friction="1.0"/>
+			<dynamics damping="0.1" friction="1.2"/>
 		</joint>
 		<!-- Right Wheel -->
@@ -312,5 +312,5 @@
 				</geometry>
 			</collision>
-			<xacro:inertial_cylinder mass="2.0" length="0.04" radius="0.09">
+			<xacro:inertial_cylinder mass="20.0" length="0.04" radius="0.09">
 				<origin xyz="0 0 0" rpy="0 0 0"/>
 			</xacro:inertial_cylinder>
@@ -332,5 +332,5 @@
 			<parent link="${prefix}right_hub"/>
 			<child link="${prefix}right_wheel"/>
-			<dynamics damping="1.0" friction="1.0"/>
+			<dynamics damping="0.1" friction="1.2"/>
 		</joint>
 		<!-- <gazebo>

Commit message: more polished

File: urdf/pioneer3dx/pioneer3dx_sim.urdf.xacro (robot description, xacro)
@@ -273,5 +273,5 @@
 			<parent link="${prefix}left_hub"/>
 			<child link="${prefix}left_wheel"/>
-			<dynamics damping="0.1" friction="1.2"/>
+			<dynamics damping="0.1" friction="1.0"/>
 		</joint>
 		<!-- Right Wheel -->
@@ -332,5 +332,5 @@
 			<parent link="${prefix}right_hub"/>
 			<child link="${prefix}right_wheel"/>
-			<dynamics damping="0.1" friction="1.2"/>
+			<dynamics damping="0.1" friction="1.0"/>
 		</joint>
 		<!-- <gazebo>
