Commit message: some constants added
urdf finished and working

fix diff drive, 1st attempt

odom restored

File: urdf/pioneer3dx/pioneer3dx_sim.urdf.xacro (robot description, xacro)
@@ -6,19 +6,40 @@
 		<link name="${prefix}base_link">
     	</link>
-		<!-- Base Link -->
+		<!-- Chassis -->
 		<xacro:property name="chassis_length" value="0.41"/>
 		<xacro:property name="chassis_width" value="0.272"/>
 		<xacro:property name="chassis_height" value="0.172"/>
+		<xacro:property name="chassis_mass" value="1.0"/>
+		<!-- Top Plate -->
+		<xacro:property name="top_plate_length" value="0.41"/>
+		<xacro:property name="top_plate_width" value="0.272"/>
+		<xacro:property name="top_plate_height" value="0.0052"/>
+		<xacro:property name="top_plate_mass" value="0.1"/>
+		<!-- Wheels -->
+		<xacro:property name="wheel_radius" value="0.009"/>
+		<xacro:property name="wheel_thickness" value="0.04"/>
+		<xacro:property name="wheel_mass" value="0.1"/>
+		<!-- Caster wheel -->
+		<xacro:property name="caster_wheel_radius" value="0.0375"/>
+		<xacro:property name="caster_wheel_thickness" value="0.01"/>
+		<xacro:property name="caster_wheel_mass" value="0.02"/>
+		<!-- Chasis -->
 		<link name="${prefix}real_base_link">
-			<xacro:inertial_box mass="30.0" x="${chassis_length}" y="${chassis_width}" z="${chassis_height}">
-            	<origin xyz="${-chassis_length/2} 0 ${chassis_height/2}" rpy="0 0 0"/>
+			<!-- <collision>
+				<origin xyz="${chassis_length/2} 0 ${chassis_height/2}"/>
+				<geometry>
+					<box size="${chassis_length} ${chassis_width} ${chassis_height}"/>
+				</geometry>
+			</collision> -->
+			<visual>
+				<origin xyz="-0.045 0 0.148" rpy="0 0 0"/>
+				<geometry>
+					<mesh filename="file://$(find amr-ros-config)/meshes/p3dx_meshes/chassis.stl"/>
+				</geometry>
+				<material name="ChassisRed"/>
+			</visual>
+			<xacro:inertial_box mass="${chassis_mass}" x="${chassis_length}" y="${chassis_width}" z="${chassis_height}">
+            	<origin xyz="${-chassis_length/2} 0 ${-chassis_height/2}" rpy="0 0 0"/>
         	</xacro:inertial_box>
-			<visual>
-				<origin xyz="-0.045 0 0.148" rpy="0 0 0"/>
-				<geometry>
-					<mesh filename="file://$(find amr-ros-config)/meshes/p3dx_meshes/chassis.stl"/>
-				</geometry>
-				<material name="ChassisRed"/>
-			</visual>
 		</link>
 		<gazebo reference="${prefix}real_base_link">
@@ -31,24 +52,21 @@
 		</joint>
 		<!-- Top Plate -->
-		<xacro:property name="top_plate_length" value="0.41"/>
-		<xacro:property name="top_plate_width" value="0.272"/>
-		<xacro:property name="top_plate_height" value="0.0052"/>
 		<link name="${prefix}top_plate">
-			<xacro:inertial_box mass="1.0" x="${top_plate_length}" y="${top_plate_width}" z="${top_plate_height}">
+			<!-- <collision>
+				<origin xyz="${top_plate_length/2} 0 ${top_plate_height/2}"/>
+				<geometry>
+					<box size="${top_plate_length} ${top_plate_width} ${top_plate_height}"/>
+				</geometry>
+			</collision> -->
+			<visual>
+				<origin xyz="0 0 0" rpy="0 0 0"/>
+				<geometry>
+					<mesh filename="file://$(find amr-ros-config)/meshes/p3dx_meshes/top.stl"/>
+				</geometry>
+				<material name="TopBlack"/>
+			</visual>
+			<xacro:inertial_box mass="${top_plate_mass}" x="${top_plate_length}" y="${top_plate_width}" z="${top_plate_height}">
             	<origin xyz="0 0 ${top_plate_height/2}" rpy="0 0 0"/>
         	</xacro:inertial_box>
-			<visual>
-				<origin xyz="0 0 0" rpy="0 0 0"/>
-				<geometry>
-					<mesh filename="file://$(find amr-ros-config)/meshes/p3dx_meshes/top.stl"/>
-				</geometry>
-				<material name="TopBlack"/>
-			</visual>
-			<collision>
-				<origin xyz="0 0 0" rpy="0 0 0"/>
-				<geometry>
-					<mesh filename="file://$(find amr-ros-config)/meshes/p3dx_meshes/top.stl"/>
-				</geometry>
-			</collision>
 		</link>
 		<gazebo reference="${prefix}top_plate">
@@ -62,4 +80,11 @@
 		<!-- Front Sonar -->
 		<link name="${prefix}front_sonar">
+			<visual>
+				<origin xyz="0 0 0" rpy="0 0 0"/>
+				<geometry>
+					<mesh filename="file://$(find amr-ros-config)/meshes/p3dx_meshes/front_sonar.stl"/>
+				</geometry>
+				<material name="SonarYellow"/>
+			</visual>
 			<inertial>
 				<mass value="0.0001"/>
@@ -67,11 +92,4 @@
 				<inertia ixx="1" ixy="0" ixz="0" iyy="1" iyz="0" izz="1"/>
 			</inertial>
-			<visual>
-				<origin xyz="0 0 0" rpy="0 0 0"/>
-				<geometry>
-					<mesh filename="file://$(find amr-ros-config)/meshes/p3dx_meshes/front_sonar.stl"/>
-				</geometry>
-				<material name="SonarYellow"/>
-			</visual>
 		</link>
 		<gazebo reference="${prefix}front_sonar">
@@ -84,10 +102,12 @@
 		</joint>
 		<!-- Back Sonar -->
-		<joint name="${prefix}base_back_joint" type="fixed">
-			<origin xyz="0.109 0 0.209" rpy="0 0 0"/>
-			<parent link="${prefix}real_base_link"/>
-			<child link="${prefix}back_sonar"/>
-		</joint>
 		<link name="${prefix}back_sonar">
+			<visual>
+				<origin xyz="0 0 0" rpy="0 0 0"/>
+				<geometry>
+					<mesh filename="file://$(find amr-ros-config)/meshes/p3dx_meshes/back_sonar.stl"/>
+				</geometry>
+				<material name="SonarYellow"/>
+			</visual>
 			<inertial>
 				<mass value="0.0001"/>
@@ -95,69 +115,64 @@
 				<inertia ixx="1" ixy="0" ixz="0" iyy="1" iyz="0" izz="1"/>
 			</inertial>
-			<visual>
-				<origin xyz="0 0 0" rpy="0 0 0"/>
-				<geometry>
-					<mesh filename="file://$(find amr-ros-config)/meshes/p3dx_meshes/back_sonar.stl"/>
-				</geometry>
-				<material name="SonarYellow"/>
-			</visual>
 		</link>
 		<gazebo reference="${prefix}back_sonar">
 			<material value="Gazebo/Yellow"/>
 		</gazebo>
+		<joint name="${prefix}base_back_joint" type="fixed">
+			<origin xyz="0.109 0 0.209" rpy="0 0 0"/>
+			<parent link="${prefix}real_base_link"/>
+			<child link="${prefix}back_sonar"/>
+		</joint>
 		<!-- Caster Swivel -->
-		<joint name="${prefix}base_caster_swivel_joint" type="continuous"> <!--Not fixed. Change for simulation -->
-			<origin xyz="-0.185 0 0.055" rpy="0 0 0"/>
-			<axis xyz="0 0 1"/>
-			<parent link="${prefix}real_base_link"/>
-			<child link="${prefix}caster_swivel"/>
-			<limit effort="10000.0" lower="-100000" upper="100000" velocity="100000"/>
-    		<!-- <dynamics damping="0.001" friction="0.0001"/> -->
-		</joint>
-		<passive_joint name="${prefix}base_caster_swivel_joint"/> <!--Not working -->
 		<link name="${prefix}caster_swivel">
+			<!-- <collision>
+				<origin xyz="0 0 0" rpy="0 0 0"/>
+				<geometry>
+					<mesh filename="file://$(find amr-ros-config)/meshes/p3dx_meshes/caster_swivel.stl"/>
+				</geometry>
+			</collision> -->
+			<visual>
+				<origin xyz="0 0 0" rpy="0 0 0"/>
+				<geometry>
+					<mesh filename="file://$(find amr-ros-config)/meshes/p3dx_meshes/caster_swivel.stl"/>
+				</geometry>
+				<material name="ChassisGrey"/>
+			</visual>
 			<inertial>
-				<mass value="0.1"/>
+				<mass value="0.01"/>
 				<origin xyz="0 0 0"/>
 				<inertia ixx="0.01" ixy="0" ixz="0" iyy="0.01" iyz="0" izz="0.01"/>
 			</inertial>
-			<visual>
-				<origin xyz="0 0 0" rpy="0 0 0"/>
-				<geometry>
-					<mesh filename="file://$(find amr-ros-config)/meshes/p3dx_meshes/caster_swivel.stl"/>
-				</geometry>
-				<material name="ChassisGrey"/>
-			</visual>
-			<!-- <collision>
-				<origin xyz="0 0 0" rpy="0 0 0"/>
-				<geometry>
-					<mesh filename="file://$(find amr-ros-config)/meshes/p3dx_meshes/caster_swivel.stl"/>
-				</geometry>
-			</collision> -->
 		</link>
 		<gazebo reference="${prefix}caster_swivel">
 			<material value="Gazebo/Grey"/>
 		</gazebo>
-		<!-- Center Wheel + Hubcap -->
+		<joint name="${prefix}base_caster_swivel_joint" type="fixed"> <!--Not fixed. Change for simulation -->
+			<origin xyz="-0.185 0 0.055" rpy="0 0 0"/>
+			<axis xyz="0 0 1"/>
+			<parent link="${prefix}real_base_link"/>
+			<child link="${prefix}caster_swivel"/>
+		</joint>
+		<!-- Hubcap -->
 		<link name="${prefix}caster_hubcap">
+			<!-- <collision>
+				<origin xyz="0 0 0" rpy="0 0 0"/>
+				<geometry>
+					<mesh filename="file://$(find amr-ros-config)/meshes/p3dx_meshes/caster_hubcap.stl"/>
+				</geometry>
+			</collision> -->
+			<visual>
+				<origin xyz="0 0 0" rpy="${1.5708} 0 0"/>
+				<geometry>
+					<mesh filename="file://$(find amr-ros-config)/meshes/p3dx_meshes/caster_hubcap.stl"/>
+				</geometry>
+				<material name="ChassisGrey"/>
+			</visual>
 			<inertial>
-				<mass value="0.1"/>
+				<mass value="0.01"/>
 				<origin xyz="0 0 0"/>
 				<inertia ixx="0.012411765597" ixy="-0.000711733678" ixz="0.00050272983"
 							iyy="0.015218160428" iyz="-0.000004273467" izz="0.011763977943"/>
 			</inertial>
-			<visual>
-				<origin xyz="0 0 0" rpy="${1.5708} 0 0"/>
-				<geometry>
-					<mesh filename="file://$(find amr-ros-config)/meshes/p3dx_meshes/caster_hubcap.stl"/>
-				</geometry>
-				<material name="ChassisGrey"/>
-			</visual>
-			<!-- <collision>
-				<origin xyz="0 0 0" rpy="0 0 0"/>
-				<geometry>
-					<mesh filename="file://$(find amr-ros-config)/meshes/p3dx_meshes/caster_hubcap.stl"/>
-				</geometry>
-			</collision> -->
 		</link>
 		<gazebo reference="${prefix}caster_hubcap">
@@ -169,36 +184,28 @@
 			<parent link="${prefix}caster_swivel"/>
 			<child link="${prefix}caster_hubcap"/>
-			<limit effort="10000.0" lower="-100000" upper="100000" velocity="100000"/>
-    		<!-- <dynamics damping="0.001" friction="0.0001"/> -->
 		</joint>
 		<!-- Caster Wheel -->
 		<link name="${prefix}caster_wheel">
-			<xacro:inertial_cylinder mass="2.0" length="0.01" radius="0.0375">
-				<origin xyz="0 0 0" rpy="0 0 0"/>
-			</xacro:inertial_cylinder>
-			<visual>
-				<origin xyz="0 0 0" rpy="0 0 0"/>
-				<geometry>
-					<cylinder radius="0.0375" length="0.01"/>
+			<collision>
+				<origin xyz="0 0 0" rpy="0 0 0"/>
+				<geometry>
+					<sphere radius="${caster_wheel_radius}"/>
+				</geometry>
+			</collision>
+			<visual>
+				<origin xyz="0 0 0" rpy="0 0 0"/>
+				<geometry>
+					<cylinder radius="${caster_wheel_radius}" length="${caster_wheel_thickness}"/>
 				</geometry>
 				<material name="WheelBlack"/>
 			</visual>
-			<collision>
-				<origin xyz="0 0 0" rpy="0 0 0"/>
-				<geometry>
-					<cylinder radius="0.0375" length="0.01"/>
-				</geometry>
-			</collision>
-			<dynamics damping="0.0001" friction="0.0001"/>
+			<xacro:inertial_cylinder mass="${caster_wheel_mass}" length="${caster_wheel_thickness}" radius="${caster_wheel_radius}">
+				<origin xyz="0 0 0" rpy="0 0 0"/>
+			</xacro:inertial_cylinder>
 		</link>
 		<gazebo reference="${prefix}caster_wheel">
 			<material value="Gazebo/White"/>
-			<kp>1000000.0</kp> <!-- kp and kd for rubber -->
-			<kd>100.0</kd>
-			<mu1>0.0</mu1>
-			<mu2>0.0</mu2>
-			<!-- fdir1 0 1 0 /fdir1 --> <!-- see http://github.com/MobileRobots/amr-ros-config/issues/6 -->
-			<maxVel>1.0</maxVel>
-			<minDepth>0.00</minDepth>
+			<mu1 value="0.001"/>
+			<mu2 value="0.001"/>
 		</gazebo>
 		<joint name="${prefix}caster_wheel_joint" type="fixed">  <!--Not fixed. Change for simulation -->
@@ -207,26 +214,23 @@
 			<parent link="${prefix}caster_hubcap"/>
 			<child link="${prefix}caster_wheel"/>
-			<dynamics damping="1.0" friction="1.0"/>
 		</joint>
 		<!-- Left Wheel -->
 		<link name="${prefix}left_hub">
-			<visual>
+			<!-- <collision>
 				<origin xyz="0 0 0" rpy="${-3.1415927/2.0} 0 0"/>
 				<geometry>
 					<cylinder radius="0.09" length="0.01"/>
 				</geometry>
+			</collision> -->
+			<visual>
+				<origin xyz="0 0 0" rpy="${-3.1415927/2.0} 0 0"/>
+				<geometry>
+					<cylinder radius="0.09" length="0.01"/>
+				</geometry>
 				<material name="HubcapYellow"/>
 			</visual>
-			<!-- <collision>
+			<xacro:inertial_cylinder mass="0.01" length="0.01" radius="0.0375">
 				<origin xyz="0 0 0" rpy="${-3.1415927/2.0} 0 0"/>
-				<geometry>
-					<cylinder radius="0.09" length="0.01"/>
-				</geometry>
-			</collision> -->
-			<inertial>
-				<mass value="0.1"/>
-				<origin xyz="0 0 0" rpy="${-3.1415927/2.0} 0 0"/>
-				<inertia ixx="0.001" ixy="0" ixz="0" iyy="0.001" iyz="0" izz="0.001"/>
-			</inertial>
+			</xacro:inertial_cylinder>
 		</link>
 		<gazebo reference="${prefix}left_hub">
@@ -240,4 +244,10 @@
 		</joint>
 		<link name="${prefix}left_wheel">
+			<collision>
+				<origin xyz="0 0 0" rpy="0 0 0"/>
+				<geometry>
+					<sphere radius="${wheel_radius}"/>
+				</geometry>
+			</collision>
 			<visual>
 				<origin xyz="0 0 0" rpy="1.5708 0 0"/>
@@ -247,24 +257,10 @@
 				<material name="WheelBlack"/>
 			</visual>
-			<collision>
-				<origin xyz="0 0 0" rpy="0 0 0"/>
-				<geometry>
-					<sphere radius="0.09"/>
-				</geometry>
-			</collision>
-			<xacro:inertial_cylinder mass="20.0" length="0.04" radius="0.09">
-				<origin xyz="0 0 0" rpy="0 0 0"/>
-			</xacro:inertial_cylinder>
-			<dynamics damping="1.0" friction="1.0"/>
+			<xacro:inertial_cylinder mass="${wheel_mass}" length="${wheel_thickness}" radius="${wheel_radius}">
+				<origin xyz="0 0 0" rpy="0 0 0"/>
+			</xacro:inertial_cylinder>
 		</link>
 		<gazebo reference="${prefix}left_wheel">
 			<material value="Gazebo/Black"/>
-			<kp>1000000.0</kp> <!-- kp and kd for rubber -->
-			<kd>100.0</kd>
-			<mu1>1.0</mu1>
-			<mu2>1.0</mu2>
-			<!-- fdir1 0 1 0 /fdir1 --> <!-- see http://github.com/MobileRobots/amr-ros-config/issues/6 -->
-			<maxVel>1.0</maxVel>
-			<minDepth>0.00</minDepth>
 		</gazebo>
 		<joint name="${prefix}left_wheel_joint" type="continuous">
@@ -273,20 +269,23 @@
 			<parent link="${prefix}left_hub"/>
 			<child link="${prefix}left_wheel"/>
-			<dynamics damping="0.1" friction="1.0"/>
 		</joint>
 		<!-- Right Wheel -->
 		<link name="${prefix}right_hub">
-			<visual>
+			<!-- <collision>
 				<origin xyz="0 0 0" rpy="${3.1415927/2.0} 0 0"/>
 				<geometry>
 					<cylinder radius="0.09" length="0.01"/>
 				</geometry>
+			</collision> -->
+			<visual>
+				<origin xyz="0 0 0" rpy="${3.1415927/2.0} 0 0"/>
+				<geometry>
+					<cylinder radius="0.09" length="0.01"/>
+				</geometry>
 				<material name="HubcapYellow"/>
 			</visual>
-			<inertial>
-				<mass value="0.1"/>
+			<xacro:inertial_cylinder mass="0.01" length="0.01" radius="0.0375">
 				<origin xyz="0 0 0" rpy="${3.1415927/2.0} 0 0"/>
-				<inertia ixx="0.001" ixy="0" ixz="0" iyy="0.001" iyz="0" izz="0.001"/>
-			</inertial>
+			</xacro:inertial_cylinder>
 		</link>
 		<gazebo reference="${prefix}right_hub">
@@ -299,4 +298,10 @@
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
Commit message: some constants added

File: urdf/pioneer3dx/pioneer3dx_sim.urdf.xacro (robot description, xacro)
@@ -6,10 +6,21 @@
 		<link name="${prefix}base_link">
     	</link>
-		<!-- Base Link -->
+		<!-- Chassis -->
 		<xacro:property name="chassis_length" value="0.41"/>
 		<xacro:property name="chassis_width" value="0.272"/>
 		<xacro:property name="chassis_height" value="0.172"/>
+		<xacro:property name="chassis_mass" value="1.0"/>
+		<!-- Wheels -->
+		<xacro:property name="wheel_radius" value="0.09"/>
+		<xacro:property name="wheel_thickness" value="0.04"/>
+		<xacro:property name="wheel_mass" value="0.05"/>
+		Caster wheels
+		<xacro:property name="caster_wheel_radius" value="0.01"/>
+		<xacro:property name="caster_wheel_mass" value="0.01"/>
+		<xacro:property name="caster_wheel_offset_x" value="0.075"/>
+		<xacro:property name="caster_wheel_offset_z" value="${wheel_offset_z - wheel_radius + caster_wheel_radius}"/>
+		<!-- Base Link -->
 		<link name="${prefix}real_base_link">
-			<xacro:inertial_box mass="30.0" x="${chassis_length}" y="${chassis_width}" z="${chassis_height}">
+			<xacro:inertial_box mass="${chassis_mass}" x="${chassis_length}" y="${chassis_width}" z="${chassis_height}">
             	<origin xyz="${-chassis_length/2} 0 ${chassis_height/2}" rpy="0 0 0"/>
         	</xacro:inertial_box>
@@ -224,9 +235,7 @@
 				</geometry>
 			</collision> -->
-			<inertial>
-				<mass value="0.1"/>
-				<origin xyz="0 0 0" rpy="${-3.1415927/2.0} 0 0"/>
-				<inertia ixx="0.001" ixy="0" ixz="0" iyy="0.001" iyz="0" izz="0.001"/>
-			</inertial>
+			<xacro:inertial_cylinder mass="2.0" length="0.01" radius="0.0375">
+				<origin xyz="0 0 0" rpy="0 0 0"/>
+			</xacro:inertial_cylinder>
 		</link>
 		<gazebo reference="${prefix}left_hub">
@@ -253,18 +262,10 @@
 				</geometry>
 			</collision>
-			<xacro:inertial_cylinder mass="20.0" length="0.04" radius="0.09">
+			<xacro:inertial_cylinder mass="0.1" length="${wheel_thickness}" radius="${wheel_radius}">
 				<origin xyz="0 0 0" rpy="0 0 0"/>
 			</xacro:inertial_cylinder>
-			<dynamics damping="1.0" friction="1.0"/>
 		</link>
 		<gazebo reference="${prefix}left_wheel">
 			<material value="Gazebo/Black"/>
-			<kp>1000000.0</kp> <!-- kp and kd for rubber -->
-			<kd>100.0</kd>
-			<mu1>1.0</mu1>
-			<mu2>1.0</mu2>
-			<!-- fdir1 0 1 0 /fdir1 --> <!-- see http://github.com/MobileRobots/amr-ros-config/issues/6 -->
-			<maxVel>1.0</maxVel>
-			<minDepth>0.00</minDepth>
 		</gazebo>
 		<joint name="${prefix}left_wheel_joint" type="continuous">
@@ -273,5 +274,4 @@
 			<parent link="${prefix}left_hub"/>
 			<child link="${prefix}left_wheel"/>
-			<dynamics damping="0.1" friction="1.0"/>
 		</joint>
 		<!-- Right Wheel -->
@@ -284,9 +284,4 @@
 				<material name="HubcapYellow"/>
 			</visual>
-			<inertial>
-				<mass value="0.1"/>
-				<origin xyz="0 0 0" rpy="${3.1415927/2.0} 0 0"/>
-				<inertia ixx="0.001" ixy="0" ixz="0" iyy="0.001" iyz="0" izz="0.001"/>
-			</inertial>
 		</link>
 		<gazebo reference="${prefix}right_hub">
@@ -312,18 +307,10 @@
 				</geometry>
 			</collision>
-			<xacro:inertial_cylinder mass="20.0" length="0.04" radius="0.09">
+			<xacro:inertial_cylinder mass="0.1" length="${wheel_thickness}" radius="${wheel_radius}">
 				<origin xyz="0 0 0" rpy="0 0 0"/>
 			</xacro:inertial_cylinder>
-			<!-- <dynamics damping="1.0" friction="1.0"/> -->
 		</link>
 		<gazebo reference="${prefix}right_wheel">
 			<material value="Gazebo/Black"/>
-			<kp>1000000.0</kp> <!-- kp and kd for rubber -->
-			<kd>100.0</kd>
-			<mu1>1.0</mu1>
-			<mu2>1.0</mu2>
-			<!-- fdir1 0 1 0 /fdir1 --> <!-- see http://github.com/MobileRobots/amr-ros-config/issues/6 -->
-			<maxVel>1.0</maxVel>
-			<minDepth>0.01</minDepth>
 		</gazebo>
 		<joint name="${prefix}right_wheel_joint" type="continuous">
@@ -332,14 +319,5 @@
 			<parent link="${prefix}right_hub"/>
 			<child link="${prefix}right_wheel"/>
-			<dynamics damping="0.1" friction="1.0"/>
-		</joint>
-		<!-- <gazebo>
-			<plugin name="ground_plane" filename="libgazebo_ros_surface_properties.so">
-				<mu>1.0</mu>
-				<mu2>1.0</mu2>
-				<kp>100000</kp>
-				<kd>1</kd>
-			</plugin>
-		</gazebo> -->
+		</joint>
 	</xacro:macro>
 </robot>
