Commit message: urdf finished and working

File: urdf/pioneer3dx/pioneer3dx_sim.urdf.xacro (robot description, xacro)
@@ -11,25 +11,34 @@
 		<xacro:property name="chassis_height" value="0.172"/>
 		<xacro:property name="chassis_mass" value="1.0"/>
+		<!-- Top Plate -->
+		<xacro:property name="top_plate_length" value="0.41"/>
+		<xacro:property name="top_plate_width" value="0.272"/>
+		<xacro:property name="top_plate_height" value="0.0052"/>
 		<!-- Wheels -->
 		<xacro:property name="wheel_radius" value="0.09"/>
 		<xacro:property name="wheel_thickness" value="0.04"/>
-		<xacro:property name="wheel_mass" value="0.05"/>
-		Caster wheels
-		<xacro:property name="caster_wheel_radius" value="0.01"/>
-		<xacro:property name="caster_wheel_mass" value="0.01"/>
-		<xacro:property name="caster_wheel_offset_x" value="0.075"/>
-		<xacro:property name="caster_wheel_offset_z" value="${wheel_offset_z - wheel_radius + caster_wheel_radius}"/>
-		<!-- Base Link -->
+		<xacro:property name="wheel_mass" value="0.1"/>
+		<!-- Caster wheel -->
+		<xacro:property name="caster_wheel_radius" value="0.0375"/>
+		<xacro:property name="caster_wheel_thickness" value="0.01"/>
+		<xacro:property name="caster_wheel_mass" value="0.02"/>
+		<!-- Chasis -->
 		<link name="${prefix}real_base_link">
+			<collision>
+				<origin xyz="${chassis_length/2} 0 ${chassis_height/2}"/>
+				<geometry>
+					<box size="${chassis_length} ${chassis_width} ${chassis_height}"/>
+				</geometry>
+			</collision>
+			<visual>
+				<origin xyz="-0.045 0 0.148" rpy="0 0 0"/>
+				<geometry>
+					<mesh filename="file://$(find amr-ros-config)/meshes/p3dx_meshes/chassis.stl"/>
+				</geometry>
+				<material name="ChassisRed"/>
+			</visual>
 			<xacro:inertial_box mass="${chassis_mass}" x="${chassis_length}" y="${chassis_width}" z="${chassis_height}">
             	<origin xyz="${-chassis_length/2} 0 ${chassis_height/2}" rpy="0 0 0"/>
         	</xacro:inertial_box>
-			<visual>
-				<origin xyz="-0.045 0 0.148" rpy="0 0 0"/>
-				<geometry>
-					<mesh filename="file://$(find amr-ros-config)/meshes/p3dx_meshes/chassis.stl"/>
-				</geometry>
-				<material name="ChassisRed"/>
-			</visual>
 		</link>
 		<gazebo reference="${prefix}real_base_link">
@@ -42,24 +51,21 @@
 		</joint>
 		<!-- Top Plate -->
-		<xacro:property name="top_plate_length" value="0.41"/>
-		<xacro:property name="top_plate_width" value="0.272"/>
-		<xacro:property name="top_plate_height" value="0.0052"/>
 		<link name="${prefix}top_plate">
+			<collision>
+				<origin xyz="${top_plate_length/2} 0 ${top_plate_height/2}"/>
+				<geometry>
+					<box size="${top_plate_length} ${top_plate_width} ${top_plate_height}"/>
+				</geometry>
+			</collision>
+			<visual>
+				<origin xyz="0 0 0" rpy="0 0 0"/>
+				<geometry>
+					<mesh filename="file://$(find amr-ros-config)/meshes/p3dx_meshes/top.stl"/>
+				</geometry>
+				<material name="TopBlack"/>
+			</visual>
 			<xacro:inertial_box mass="1.0" x="${top_plate_length}" y="${top_plate_width}" z="${top_plate_height}">
             	<origin xyz="0 0 ${top_plate_height/2}" rpy="0 0 0"/>
         	</xacro:inertial_box>
-			<visual>
-				<origin xyz="0 0 0" rpy="0 0 0"/>
-				<geometry>
-					<mesh filename="file://$(find amr-ros-config)/meshes/p3dx_meshes/top.stl"/>
-				</geometry>
-				<material name="TopBlack"/>
-			</visual>
-			<collision>
-				<origin xyz="0 0 0" rpy="0 0 0"/>
-				<geometry>
-					<mesh filename="file://$(find amr-ros-config)/meshes/p3dx_meshes/top.stl"/>
-				</geometry>
-			</collision>
 		</link>
 		<gazebo reference="${prefix}top_plate">
@@ -73,4 +79,11 @@
 		<!-- Front Sonar -->
 		<link name="${prefix}front_sonar">
+			<visual>
+				<origin xyz="0 0 0" rpy="0 0 0"/>
+				<geometry>
+					<mesh filename="file://$(find amr-ros-config)/meshes/p3dx_meshes/front_sonar.stl"/>
+				</geometry>
+				<material name="SonarYellow"/>
+			</visual>
 			<inertial>
 				<mass value="0.0001"/>
@@ -78,11 +91,4 @@
 				<inertia ixx="1" ixy="0" ixz="0" iyy="1" iyz="0" izz="1"/>
 			</inertial>
-			<visual>
-				<origin xyz="0 0 0" rpy="0 0 0"/>
-				<geometry>
-					<mesh filename="file://$(find amr-ros-config)/meshes/p3dx_meshes/front_sonar.stl"/>
-				</geometry>
-				<material name="SonarYellow"/>
-			</visual>
 		</link>
 		<gazebo reference="${prefix}front_sonar">
@@ -95,10 +101,12 @@
 		</joint>
 		<!-- Back Sonar -->
-		<joint name="${prefix}base_back_joint" type="fixed">
-			<origin xyz="0.109 0 0.209" rpy="0 0 0"/>
-			<parent link="${prefix}real_base_link"/>
-			<child link="${prefix}back_sonar"/>
-		</joint>
 		<link name="${prefix}back_sonar">
+			<visual>
+				<origin xyz="0 0 0" rpy="0 0 0"/>
+				<geometry>
+					<mesh filename="file://$(find amr-ros-config)/meshes/p3dx_meshes/back_sonar.stl"/>
+				</geometry>
+				<material name="SonarYellow"/>
+			</visual>
 			<inertial>
 				<mass value="0.0001"/>
@@ -106,69 +114,64 @@
 				<inertia ixx="1" ixy="0" ixz="0" iyy="1" iyz="0" izz="1"/>
 			</inertial>
-			<visual>
-				<origin xyz="0 0 0" rpy="0 0 0"/>
-				<geometry>
-					<mesh filename="file://$(find amr-ros-config)/meshes/p3dx_meshes/back_sonar.stl"/>
-				</geometry>
-				<material name="SonarYellow"/>
-			</visual>
 		</link>
 		<gazebo reference="${prefix}back_sonar">
 			<material value="Gazebo/Yellow"/>
 		</gazebo>
+		<joint name="${prefix}base_back_joint" type="fixed">
+			<origin xyz="0.109 0 0.209" rpy="0 0 0"/>
+			<parent link="${prefix}real_base_link"/>
+			<child link="${prefix}back_sonar"/>
+		</joint>
 		<!-- Caster Swivel -->
-		<joint name="${prefix}base_caster_swivel_joint" type="continuous"> <!--Not fixed. Change for simulation -->
-			<origin xyz="-0.185 0 0.055" rpy="0 0 0"/>
-			<axis xyz="0 0 1"/>
-			<parent link="${prefix}real_base_link"/>
-			<child link="${prefix}caster_swivel"/>
-			<limit effort="10000.0" lower="-100000" upper="100000" velocity="100000"/>
-    		<!-- <dynamics damping="0.001" friction="0.0001"/> -->
-		</joint>
-		<passive_joint name="${prefix}base_caster_swivel_joint"/> <!--Not working -->
 		<link name="${prefix}caster_swivel">
+			<!-- <collision>
+				<origin xyz="0 0 0" rpy="0 0 0"/>
+				<geometry>
+					<mesh filename="file://$(find amr-ros-config)/meshes/p3dx_meshes/caster_swivel.stl"/>
+				</geometry>
+			</collision> -->
+			<visual>
+				<origin xyz="0 0 0" rpy="0 0 0"/>
+				<geometry>
+					<mesh filename="file://$(find amr-ros-config)/meshes/p3dx_meshes/caster_swivel.stl"/>
+				</geometry>
+				<material name="ChassisGrey"/>
+			</visual>
 			<inertial>
-				<mass value="0.1"/>
+				<mass value="0.01"/>
 				<origin xyz="0 0 0"/>
 				<inertia ixx="0.01" ixy="0" ixz="0" iyy="0.01" iyz="0" izz="0.01"/>
 			</inertial>
-			<visual>
-				<origin xyz="0 0 0" rpy="0 0 0"/>
-				<geometry>
-					<mesh filename="file://$(find amr-ros-config)/meshes/p3dx_meshes/caster_swivel.stl"/>
-				</geometry>
-				<material name="ChassisGrey"/>
-			</visual>
-			<!-- <collision>
-				<origin xyz="0 0 0" rpy="0 0 0"/>
-				<geometry>
-					<mesh filename="file://$(find amr-ros-config)/meshes/p3dx_meshes/caster_swivel.stl"/>
-				</geometry>
-			</collision> -->
 		</link>
 		<gazebo reference="${prefix}caster_swivel">
 			<material value="Gazebo/Grey"/>
 		</gazebo>
-		<!-- Center Wheel + Hubcap -->
+		<joint name="${prefix}base_caster_swivel_joint" type="continuous"> <!--Not fixed. Change for simulation -->
+			<origin xyz="-0.185 0 0.055" rpy="0 0 0"/>
+			<axis xyz="0 0 1"/>
+			<parent link="${prefix}real_base_link"/>
+			<child link="${prefix}caster_swivel"/>
+		</joint>
+		<!-- Hubcap -->
 		<link name="${prefix}caster_hubcap">
+			<!-- <collision>
+				<origin xyz="0 0 0" rpy="0 0 0"/>
+				<geometry>
+					<mesh filename="file://$(find amr-ros-config)/meshes/p3dx_meshes/caster_hubcap.stl"/>
+				</geometry>
+			</collision> -->
+			<visual>
+				<origin xyz="0 0 0" rpy="${1.5708} 0 0"/>
+				<geometry>
+					<mesh filename="file://$(find amr-ros-config)/meshes/p3dx_meshes/caster_hubcap.stl"/>
+				</geometry>
+				<material name="ChassisGrey"/>
+			</visual>
 			<inertial>
-				<mass value="0.1"/>
+				<mass value="0.01"/>
 				<origin xyz="0 0 0"/>
 				<inertia ixx="0.012411765597" ixy="-0.000711733678" ixz="0.00050272983"
 							iyy="0.015218160428" iyz="-0.000004273467" izz="0.011763977943"/>
 			</inertial>
-			<visual>
-				<origin xyz="0 0 0" rpy="${1.5708} 0 0"/>
-				<geometry>
-					<mesh filename="file://$(find amr-ros-config)/meshes/p3dx_meshes/caster_hubcap.stl"/>
-				</geometry>
-				<material name="ChassisGrey"/>
-			</visual>
-			<!-- <collision>
-				<origin xyz="0 0 0" rpy="0 0 0"/>
-				<geometry>
-					<mesh filename="file://$(find amr-ros-config)/meshes/p3dx_meshes/caster_hubcap.stl"/>
-				</geometry>
-			</collision> -->
 		</link>
 		<gazebo reference="${prefix}caster_hubcap">
@@ -180,36 +183,28 @@
 			<parent link="${prefix}caster_swivel"/>
 			<child link="${prefix}caster_hubcap"/>
-			<limit effort="10000.0" lower="-100000" upper="100000" velocity="100000"/>
-    		<!-- <dynamics damping="0.001" friction="0.0001"/> -->
 		</joint>
 		<!-- Caster Wheel -->
 		<link name="${prefix}caster_wheel">
-			<xacro:inertial_cylinder mass="2.0" length="0.01" radius="0.0375">
-				<origin xyz="0 0 0" rpy="0 0 0"/>
-			</xacro:inertial_cylinder>
-			<visual>
-				<origin xyz="0 0 0" rpy="0 0 0"/>
-				<geometry>
-					<cylinder radius="0.0375" length="0.01"/>
+			<collision>
+				<origin xyz="0 0 0" rpy="0 0 0"/>
+				<geometry>
+					<sphere radius="${caster_wheel_radius}"/>
+				</geometry>
+			</collision>
+			<visual>
+				<origin xyz="0 0 0" rpy="0 0 0"/>
+				<geometry>
+					<cylinder radius="${caster_wheel_radius}" length="${caster_wheel_thickness}"/>
 				</geometry>
 				<material name="WheelBlack"/>
 			</visual>
-			<collision>
-				<origin xyz="0 0 0" rpy="0 0 0"/>
-				<geometry>
-					<cylinder radius="0.0375" length="0.01"/>
-				</geometry>
-			</collision>
-			<dynamics damping="0.0001" friction="0.0001"/>
+			<xacro:inertial_cylinder mass="${caster_wheel_mass}" length="${caster_wheel_thickness}" radius="${caster_wheel_radius}">
+				<origin xyz="0 0 0" rpy="0 0 0"/>
+			</xacro:inertial_cylinder>
 		</link>
 		<gazebo reference="${prefix}caster_wheel">
 			<material value="Gazebo/White"/>
-			<kp>1000000.0</kp> <!-- kp and kd for rubber -->
-			<kd>100.0</kd>
-			<mu1>0.0</mu1>
-			<mu2>0.0</mu2>
-			<!-- fdir1 0 1 0 /fdir1 --> <!-- see http://github.com/MobileRobots/amr-ros-config/issues/6 -->
-			<maxVel>1.0</maxVel>
-			<minDepth>0.00</minDepth>
+			<mu1 value="0.001"/>
+			<mu2 value="0.001"/>
 		</gazebo>
 		<joint name="${prefix}caster_wheel_joint" type="fixed">  <!--Not fixed. Change for simulation -->
@@ -218,15 +213,7 @@
 			<parent link="${prefix}caster_hubcap"/>
 			<child link="${prefix}caster_wheel"/>
-			<dynamics damping="1.0" friction="1.0"/>
 		</joint>
 		<!-- Left Wheel -->
 		<link name="${prefix}left_hub">
-			<visual>
-				<origin xyz="0 0 0" rpy="${-3.1415927/2.0} 0 0"/>
-				<geometry>
-					<cylinder radius="0.09" length="0.01"/>
-				</geometry>
-				<material name="HubcapYellow"/>
-			</visual>
 			<!-- <collision>
 				<origin xyz="0 0 0" rpy="${-3.1415927/2.0} 0 0"/>
@@ -235,6 +222,13 @@
 				</geometry>
 			</collision> -->
-			<xacro:inertial_cylinder mass="2.0" length="0.01" radius="0.0375">
-				<origin xyz="0 0 0" rpy="0 0 0"/>
+			<visual>
+				<origin xyz="0 0 0" rpy="${-3.1415927/2.0} 0 0"/>
+				<geometry>
+					<cylinder radius="0.09" length="0.01"/>
+				</geometry>
+				<material name="HubcapYellow"/>
+			</visual>
+			<xacro:inertial_cylinder mass="0.01" length="0.01" radius="0.0375">
+				<origin xyz="0 0 0" rpy="${-3.1415927/2.0} 0 0"/>
 			</xacro:inertial_cylinder>
 		</link>
@@ -249,4 +243,10 @@
 		</joint>
 		<link name="${prefix}left_wheel">
+			<collision>
+				<origin xyz="0 0 0" rpy="0 0 0"/>
+				<geometry>
+					<sphere radius="${wheel_radius}"/>
+				</geometry>
+			</collision>
 			<visual>
 				<origin xyz="0 0 0" rpy="1.5708 0 0"/>
@@ -256,11 +256,5 @@
 				<material name="WheelBlack"/>
 			</visual>
-			<collision>
-				<origin xyz="0 0 0" rpy="0 0 0"/>
-				<geometry>
-					<sphere radius="0.09"/>
-				</geometry>
-			</collision>
-			<xacro:inertial_cylinder mass="0.1" length="${wheel_thickness}" radius="${wheel_radius}">
+			<xacro:inertial_cylinder mass="${wheel_mass}" length="${wheel_thickness}" radius="${wheel_radius}">
 				<origin xyz="0 0 0" rpy="0 0 0"/>
 			</xacro:inertial_cylinder>
@@ -277,11 +271,20 @@
 		<!-- Right Wheel -->
 		<link name="${prefix}right_hub">
-			<visual>
+			<!-- <collision>
 				<origin xyz="0 0 0" rpy="${3.1415927/2.0} 0 0"/>
 				<geometry>
 					<cylinder radius="0.09" length="0.01"/>
 				</geometry>
+			</collision> -->
+			<visual>
+				<origin xyz="0 0 0" rpy="${3.1415927/2.0} 0 0"/>
+				<geometry>
+					<cylinder radius="0.09" length="0.01"/>
+				</geometry>
 				<material name="HubcapYellow"/>
 			</visual>
+			<xacro:inertial_cylinder mass="0.01" length="0.01" radius="0.0375">
+				<origin xyz="0 0 0" rpy="${3.1415927/2.0} 0 0"/>
+			</xacro:inertial_cylinder>
 		</link>
 		<gazebo reference="${prefix}right_hub">
@@ -294,4 +297,10 @@
 		</joint>
 		<link name="${prefix}right_wheel">
+			<collision>
+				<origin xyz="0 0 0" rpy="0 0 0"/>
+				<geometry>
+					<sphere radius="${wheel_radius}"/>
+				</geometry>
+			</collision>
 			<visual>
 				<origin xyz="0 0 0" rpy="-1.5708 0 0"/>
@@ -301,11 +310,5 @@
 				<material name="WheelBlack"/>
 			</visual>
-			<collision>
-				<origin xyz="0 0 0" rpy="0 0 0"/>
-				<geometry>
-					<sphere radius="0.09"/>
-				</geometry>
-			</collision>
-			<xacro:inertial_cylinder mass="0.1" length="${wheel_thickness}" radius="${wheel_radius}">
+			<xacro:inertial_cylinder mass="${wheel_mass}" length="${wheel_thickness}" radius="${wheel_radius}">
 				<origin xyz="0 0 0" rpy="0 0 0"/>
 			</xacro:inertial_cylinder>

Commit message: last optimization

File: urdf/pioneer3dx/pioneer3dx_sim.urdf.xacro (robot description, xacro)
@@ -17,5 +17,5 @@
 		<xacro:property name="top_plate_mass" value="0.1"/>
 		<!-- Wheels -->
-		<xacro:property name="wheel_radius" value="0.009"/>
+		<xacro:property name="wheel_radius" value="0.09"/>
 		<xacro:property name="wheel_thickness" value="0.04"/>
 		<xacro:property name="wheel_mass" value="0.1"/>
@@ -40,5 +40,5 @@
 			</visual>
 			<xacro:inertial_box mass="${chassis_mass}" x="${chassis_length}" y="${chassis_width}" z="${chassis_height}">
-            	<origin xyz="${-chassis_length/2} 0 ${-chassis_height/2}" rpy="0 0 0"/>
+            	<origin xyz="${-chassis_length} 0 ${-chassis_height}" rpy="0 0 0"/>
         	</xacro:inertial_box>
 		</link>
@@ -319,6 +319,6 @@
 		</gazebo>
 		<joint name="${prefix}right_wheel_joint" type="continuous">
-			<origin xyz="0 0 0" rpy="-1.5708 0 0"/>
-			<axis xyz="0 0 1"/>
+			<origin xyz="0 0 0" rpy="1.5708 0 0"/>
+			<axis xyz="0 0 -1"/>
 			<parent link="${prefix}right_hub"/>
 			<child link="${prefix}right_wheel"/>
